File: DESIGN FILES/mux_io_tft.kicad_sch (KiCad schematic)
At the start: 0 parts

Commit message: updates
Parts:
- added C?: 47uF, soundsom:CL21A476MQYNNNE_0805, symbol soundsom:CL21A476MQYNNNE
- added C?: 100nF, soundsom:CC0603KRX7R9BB104_0603, symbol soundsom:CC0603KRX7R9BB104
- added FB?: 600R, soundsom:UPZ1608U601-1R3TF_0603, symbol soundsom:UPZ1608U601-1R3TF
- added J?: TSW-124-08-G-D, soundsom:TSW-124-08-G-D, symbol soundsom:TSW-124-08-G-D
- added J?: Micro SD, soundsom:TF-15x15_smd, symbol soundsom:TF-15x15
- added R?: 0R, soundsom:0603WAF0000T5E_0603, symbol soundsom:0603WAF0000T5E
- added R? (x5): 47k, soundsom:0603WAF4702T5E_0603, symbol soundsom:0603WAF4702T5E
- added U?: CD74HC4067, soundsom:CD74HC4067_SOIC-24, symbol soundsom:CD74HC4067
Connections:
- new net: J?.1 (DAT2), R?.2
- new net: J?.8 (DAT1), R?.2
- new net +3V3: C?.2, FB?.1, J?.01, J?.02, J?.03, J?.04, J?.37, J?.39, R?.1, R?.1, R?.1, R?.1, R?.1, U?.24 (VCC)
- new net AUXL: J?.14
- new net AUXR: J?.15
- new net CLK: J?.5 (CLK), R?.2
- new net GND: C?.1, C?.2, J?.10 (MP1), J?.11 (MP2), J?.12 (MP3), J?.13 (MP4), J?.45, J?.47, J?.48, J?.6 (VSS), U?.12 (GND), U?.15 (~{E})
- new net I34: J?.44
- new net I35: J?.41
- new net I36: J?.46
- new net I39: J?.43
- new net IO12/MUX_S2: U?.14 (S2)
- new net IO15/MUX_COM: U?.1 (COM)
- new net IO18/SD_CLK: R?.1
- new net IO19/SD_MISO: J?.7 (DAT0), R?.2
- new net IO23/SD_MOSI: J?.3 (CMD), R?.2
- new net IO2/MUX_S0: U?.10 (S0)
- new net IO32/MUX_S3: U?.13 (S3)
- new net IO4/MUX_S1: U?.11 (S1)
- new net IO5/SD_CS: J?.2 (DAT3/CD), R?.2
- new net L2: J?.10
- new net LIN: J?.09
- new net LIP: J?.08
- new net LOUT1: J?.06
- new net LOUT2: J?.20
- new net MICBIAS: J?.07
- new net MIDI_IN_RING: J?.35
- new net MIDI_IN_TIP: J?.38
- new net MUX_IO0: J?.19, U?.9 (I0)
- new net MUX_IO1: J?.22, U?.8 (I1)
- new net MUX_IO10: J?.34, U?.21 (I10)
- new net MUX_IO11: J?.31, U?.20 (I11)
- new net MUX_IO12: J?.32, U?.19 (I12)
- new net MUX_IO13: J?.29, U?.18 (I13)
- new net MUX_IO14: J?.30, U?.17 (I14)
- new net MUX_IO15: J?.27, U?.16 (I15)
- new net MUX_IO2: J?.21, U?.7 (I2)
- new net MUX_IO3: J?.24, U?.6 (I3)
- new net MUX_IO4: J?.23, U?.5 (I4)
- new net MUX_IO5: J?.26, U?.4 (I5)
- new net MUX_IO6: J?.25, U?.3 (I6)
- new net MUX_IO7: J?.28, U?.2 (I7)
- new net MUX_IO8: J?.36, U?.23 (I8)
- new net MUX_IO9: J?.33, U?.22 (I9)
- new net OUT: J?.42
- new net OUT3: J?.17
- new net OUT4: J?.16
- new net R2: J?.13
- new net RIN: J?.12
- new net RIP: J?.11
- new net ROUT1: J?.05
- new net ROUT2: J?.18
- new net SD_VDD: C?.1, FB?.2, J?.4 (VDD)
- new net THRU: J?.40
Other:
- note added: "0R : for damping resistor value testing"
- note added: "2x27 IO BUS"
- note added: "HC 3V3 OK HCT 3V3 NOK"
- note added: "MICRO SD"
- note added: "MULTIPLEXER"
