File: DESIGN FILES/ESP32 synth.kicad_sch (KiCad schematic)
At the start: 0 parts

Commit message: updates
Parts:
- added H? (x4): MountingHole, MountingHole:MountingHole_2.5mm_Pad, symbol Mechanical:MountingHole
Other:
- sheet MCU - USB - JTA renamed MCU - USB - JTAG
- company: (none) -> SOLAR AUDIO
- title: (none) -> SOLAR AUDIO - Little Sun

Commit message: updates
Other:
- sheet MUX - IO - TFT renamed MUX - POTS
- added sheet SD - TFT (sd_tft.kicad_sch)
- note added: "MOUNTING HOLES"
- note added: "PAGE 8"
- moved on the sheet: H?

Commit message: updates
Parts:
- gave numbers to parts that had none: 4
Other:
- sheet MUX - POTS: file mux_io_tft.kicad_sch -> mux_pots.kicad_sch

Commit message: updates
Other:
- sheet MCU - USB - JTAG renamed MCU - USB
- removed sheet SD - TFT
- sheet MCU - USB: file mcu_usb_jtag.kicad_sch -> mcu_usb.kicad_sch
- note removed: "PAGE 8"
- moved on the sheet: H101, H102, H103, H104
