File: DESIGN FILES/mux_pots.kicad_sch (KiCad schematic)
At the start: 19 parts, among them U701 CD74HC4067

Commit message: updates
Other:
- note added: "MUX - POTS"
- company: (none) -> Joël Ucedo
- title: (none) -> ESP32 SYNTH
- moved on the sheet: C701, RV701, RV702, RV703, RV704, RV705, RV706, RV707, RV708, RV709, RV710, RV711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

Commit message: updates
Connections:
- net MUX_IO12: now also RV715.2; no longer RV711.2
- net MUX_IO13: now also RV711.2; no longer RV715.2
- net MUX_IO2: now also RV707.2; no longer RV703.2
- net MUX_IO3: now also RV703.2; no longer RV707.2
Changed lines of the file:
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@@
     )
   )
-  (global_label "MUX_IO13" (shape input) (at 189.23 152.4 0) (fields_autoplaced)
+  (global_label "MUX_IO12" (shape input) (at 189.23 152.4 0) (fields_autoplaced)
     (effects (font (size 1.27 1.27) bold italic) (justify left))
     (property "Intersheet References" "${INTERSHEET_REFS}" (id 0) (at 201.4024 152.273 0)
@@
     )
   )
-  (global_label "MUX_IO3" (shape input) (at 123.19 152.4 0) (fields_autoplaced)
+  (global_label "MUX_IO2" (shape input) (at 123.19 152.4 0) (fields_autoplaced)
     (effects (font (size 1.27 1.27) bold italic) (justify left))
     (property "Intersheet References" "${INTERSHEET_REFS}" (id 0) (at 134.1529 152.273 0)
@@
     )
   )
-  (global_label "MUX_IO2" (shape input) (at 92.71 152.4 0) (fields_autoplaced)
+  (global_label "MUX_IO3" (shape input) (at 92.71 152.4 0) (fields_autoplaced)
     (effects (font (size 1.27 1.27) bold italic) (justify left))
     (property "Intersheet References" "${INTERSHEET_REFS}" (id 0) (at 103.6729 152.273 0)
@@
     )
   )
-  (global_label "MUX_IO12" (shape input) (at 156.21 152.4 0) (fields_autoplaced)
+  (global_label "MUX_IO13" (shape input) (at 156.21 152.4 0) (fields_autoplaced)
     (effects (font (size 1.27 1.27) bold italic) (justify left))
     (property "Intersheet References" "${INTERSHEET_REFS}" (id 0) (at 168.3824 152.273 0)

Commit message: updates
Connections:
- net IO27/MUX_S1 renamed IO32/MUX_S1
Changed lines of the file:
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@@
+    )
+  )
+  (global_label "IO32{slash}MUX_S1" (shape input) (at 306.07 139.7 180) (fields_autoplaced)
+    (effects (font (size 1.27 1.27) (thickness 0.254) bold italic) (justify right))
+    (property "Intersheet References" "${INTERSHEET_REFS}" (id 0) (at 290.1481 139.827 0)
+      (effects (font (size 1.27 1.27) (thickness 0.254) bold italic) (justify right) hide)
     )
   )
@@
     )
   )
-  (global_label "IO27{slash}MUX_S1" (shape input) (at 306.07 139.7 180) (fields_autoplaced)
-    (effects (font (size 1.27 1.27) (thickness 0.254) bold italic) (justify right))
-    (property "Intersheet References" "${INTERSHEET_REFS}" (id 0) (at 290.1481 139.827 0)
-      (effects (font (size 1.27 1.27) (thickness 0.254) bold italic) (justify right) hide)
-    )
-  )
