File: DESIGN FILES/sd_tft.kicad_sch (KiCad schematic)
At the start: 0 parts

Commit message: updates
Parts:
- added C801: 22u, MY CAPACITOR LIBRARY:0603_CL10A226MQ8NRNC, symbol MY CAPACITOR LIBRARY:CL10A226MQ8NRNC
- added FB801: 600R, MY FERRITE BEAD LIBRARY:UPZ1608U601-1R3TF_0603, symbol MY FERRITE BEAD LIBRARY:UPZ1608U601-1R3TF
- added J801: TF-15x15, MY CONNECTOR LIBRARY:TF-15x15_smd, symbol MY CONNECTOR LIBRARY:TF-15x15
- added J802: TFT-LCD, MY CONNECTOR LIBRARY:801-87-008-10-003101, symbol MY CONNECTOR LIBRARY:801-87-008-10-003101
- added R801, R802, R803, R804, R805: 47k, MY RESISTOR LIBRARY:0603WAF4702T5E, symbol MY RESISTOR LIBRARY:0603WAF4702T5E
Connections:
- new net: J801.1 (DAT2), R805.2
- new net: J801.8 (DAT1), R801.2
- new net +3V3: FB801.1, R801.1, R802.1, R803.1, R804.1, R805.1
- new net GND: C801.2, J801.10 (MP1), J801.11 (MP2), J801.12 (MP3), J801.13 (MP4), J801.6 (VSS)
- new net IO18/SD_CLK: J801.5 (CLK)
- new net IO19/SD_MISO: J801.7 (DAT0), R802.2
- new net IO23/SD_MOSI: J801.3 (CMD), R803.2
- new net IO5/SD_CS: J801.2 (DAT3/CD), R804.2
- new net SD_VDD: C801.1, FB801.2, J801.4 (VDD)
- no-connect marks 0 -> 1
Other:
- note added: "0R : for damping resistor value testing"
- note added: "MICRO SD"
- note added: "TFT-LCD"

Commit message: updates
Connections:
- net +3V3: now also J802.7 (Pin_7)
- net GND: now also J802.8 (Pin_8)
Changed lines of the file:
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@@
+    (stroke (width 0) (type default) (color 0 0 0 0))
+  )
+  (wire (pts (xy 271.78 160.02) (xy 274.32 160.02))
     (stroke (width 0) (type default) (color 0 0 0 0))
   )
@@
   )
   (wire (pts (xy 127 146.05) (xy 127 137.16))
-    (stroke (width 0) (type default) (color 0 0 0 0))
-  )
-  (wire (pts (xy 271.78 162.56) (xy 292.1 162.56))
     (stroke (width 0) (type default) (color 0 0 0 0))
   )
@@
     (stroke (width 0) (type default) (color 0 0 0 0))
   )
+  (wire (pts (xy 274.32 162.56) (xy 271.78 162.56))
+    (stroke (width 0) (type default) (color 0 0 0 0))
+  )
   (wire (pts (xy 100.33 137.16) (xy 100.33 161.29))
     (stroke (width 0) (type default) (color 0 0 0 0))
@@
   )
   (wire (pts (xy 134.62 176.53) (xy 134.62 181.61))
+    (stroke (width 0) (type default) (color 0 0 0 0))
+  )
+  (wire (pts (xy 274.32 165.1) (xy 274.32 162.56))
     (stroke (width 0) (type default) (color 0 0 0 0))
   )
@@
   )
   (wire (pts (xy 91.44 163.83) (xy 138.43 163.83))
-    (stroke (width 0) (type default) (color 0 0 0 0))
-  )
-  (wire (pts (xy 271.78 160.02) (xy 292.1 160.02))
     (stroke (width 0) (type default) (color 0 0 0 0))
   )
@@
     (pin "1")
     (pin "2")
+  )
+  (symbol (lib_id "power:+3V3") (at 274.32 160.02 270) (unit 1)
+    (in_bom yes) (on_board yes)
+    (property "Reference" "#PWR?" (id 0) (at 270.51 160.02 0)
+      (effects (font (size 1.27 1.27)) hide)
+    )
+    (property "Value" "+3V3" (id 1) (at 280.67 160.02 90))
+    (property "Footprint" "" (id 2) (at 274.32 160.02 0)
+      (effects (font (size 1.27 1.27)) hide)
+    )
+    (property "Datasheet" "" (id 3) (at 274.32 160.02 0)
+      (effects (font (size 1.27 1.27)) hide)
+    )
+    (pin "1")
   )
   (symbol (lib_id "MY CONNECTOR LIBRARY:TF-15x15") (at 162.56 161.29 0) (unit 1)
@@
     (pin "2")
   )
+  (symbol (lib_id "power:GND") (at 274.32 165.1 0) (unit 1)
+    (in_bom yes) (on_board yes) (fields_autoplaced)
+    (property "Reference" "#PWR?" (id 0) (at 274.32 171.45 0)
+      (effects (font (size 1.27 1.27)) hide)
+    )
+    (property "Value" "GND" (id 1) (at 274.32 170.18 0))
+    (property "Footprint" "" (id 2) (at 274.32 165.1 0)
+      (effects (font (size 1.27 1.27)) hide)
+    )
+    (property "Datasheet" "" (id 3) (at 274.32 165.1 0)
+      (effects (font (size 1.27 1.27)) hide)
+    )
+    (pin "1")
+  )
   (symbol (lib_id "power:GND") (at 134.62 181.61 0) (unit 1)
