File: DESIGN FILES/block_diagram.kicad_sch (KiCad schematic)
At the start: 0 parts

Commit message: updates
Other:
- note added: "BLOCK DIAGRAM"
- company: (none) -> Joël Ucedo
- title: (none) -> ESP32 SYNTH
Changed lines of the file:
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@@
 (kicad_sch (version 20211123) (generator eeschema)
-  (paper "A4")
+  (paper "A3")
+  (title_block
+    (title "ESP32 SYNTH")
+    (date "2023-06-02")
+    (rev "0")
+    (company "Joël Ucedo")
+  )
+  (text "BLOCK DIAGRAM" (at 25.4 31.75 0)
+    (effects (font (size 10 10) bold italic) (justify left bottom))
+  )
 )
