File: DESIGN FILES/audio.kicad_sch (KiCad schematic)
At the start: 0 parts

Commit message: updates
Parts:
- added C? (x5): 4.7uF, soundsom:CL10A475KO8NNNC_0603, symbol soundsom:CL10A475KO8NNNC
- added R? (x3): 0R, soundsom:0603WAF0000T5E_0603, symbol soundsom:0603WAF0000T5E
- added R?: 10k, soundsom:0603WAF1002T5E_0603, symbol soundsom:0603WAF1002T5E
- added R? (x2): 2.2k, soundsom:0603WAF2201T5E_0603, symbol soundsom:0603WAF2201T5E
- added U?: WM8978CGEFL/RV, soundsom:WM8978CGEFL_RV_WQFN-32, symbol soundsom:WM8978CGEFL{brace}slash}RV
Connections:
- new net: R?.1, U?.18 (MODE)
- new net +3.3VA: C?.1, U?.31 (AVDD)
- new net +3V3: C?.1, C?.1, R?.1, R?.1, U?.13 (DCVDD), U?.14 (DBVDD)
- new net +5V: C?.1, U?.26 (SPKVDD)
- new net AUXL: U?.19 (AUXL)
- new net AUXR: U?.20 (AUXR)
- new net BCLK: R?.2, U?.8 (BCLK)
- new net GND: C?.2, C?.2, C?.2, C?.2, C?.2, R?.2, U?.12 (DGND), U?.24 (SPKGND), U?.28 (AGND), U?.33 (AGND)
- new net IO0/MCLK: R?.1
- new net IO21/CODEC_SDIN: R?.2, U?.17 (SDIN)
- new net IO22/CODEC_SCLK: R?.2, U?.16 (SCLK)
- new net IO25/LRC: R?.1
- new net IO26/DACDAT: U?.10 (DACDAT)
- new net IO27/ADCDAT: U?.9 (ADCDAT)
- new net IO33/BCLK: R?.1
- new net L2: U?.3 (L2/GPIO2)
- new net LIN: U?.2 (LIN)
- new net LIP: U?.1 (LIP)
- new net LOUT1: U?.30 (LOUT1)
- new net LOUT2: U?.25 (LOUT2)
- new net LRC: R?.2, U?.7 (LRC)
- new net MCLK: R?.2, U?.11 (MCLK)
- new net MICBIAS: U?.32 (MICBIAS)
- new net OUT3: U?.22 (OUT3)
- new net OUT4: U?.21 (OUT4)
- new net R2: U?.6 (R2/GPIO3)
- new net RIN: U?.5 (RIN)
- new net RIP: U?.4 (RIP)
- new net ROUT1: U?.29 (ROUT1)
- new net ROUT2: U?.23 (ROUT2)
- new net VMID: C?.1, U?.27 (VMID)
- no-connect marks 0 -> 1
Other:
- note added: "0R : for damping resistor value testing"
- note added: "AUDIO CODEC"
- note added: "AVDD"
- note added: "DBVDD"
- note added: "DCVDD"
- note added: "DECOUPLING"
- note added: "I2C"
- note added: "SPKVDD"

Commit message: updates
Parts:
- removed C? (x5): 4.7uF, soundsom:CL10A475KO8NNNC_0603, symbol soundsom:CL10A475KO8NNNC
- removed R? (x3): 0R, soundsom:0603WAF0000T5E_0603, symbol soundsom:0603WAF0000T5E
- removed R?: 10k, soundsom:0603WAF1002T5E_0603, symbol soundsom:0603WAF1002T5E
- removed R? (x2): 2.2k, soundsom:0603WAF2201T5E_0603, symbol soundsom:0603WAF2201T5E
- removed U?: WM8978CGEFL/RV, soundsom:WM8978CGEFL_RV_WQFN-32, symbol soundsom:WM8978CGEFL{brace}slash}RV
- added C501, C502, C503, C504, C505: 4.7u, MY CAPACITOR LIBRARY:CL10A475KO8NNNC_0603, symbol MY CAPACITOR LIBRARY:CL10A475KO8NNNC
- added C506, C507, C510, C511: 1u, MY CAPACITOR LIBRARY:CL10A105KB8NNNC_0603, symbol MY CAPACITOR LIBRARY:CL10A105KB8NNNC
- added C508, C509: 220u, MY CAPACITOR LIBRARY:RVT1A221M0605, symbol MY CAPACITOR LIBRARY:RVT1A221M0605
- added J501, J502, J503: PJ-342B-TX-SMT, MY CONNECTOR LIBRARY:PJ-342B-TX-SMT, symbol MY CONNECTOR LIBRARY:PJ-342B-TX-SMT
- added R501, R502: 2.2k, MY RESISTOR LIBRARY:0603WAF2201T5E, symbol MY RESISTOR LIBRARY:0603WAF2201T5E
- added R503: 10k, MY RESISTOR LIBRARY:0603WAF1002T5E, symbol MY RESISTOR LIBRARY:0603WAF1002T5E
- added R504, R505: 100R, MY RESISTOR LIBRARY:0805W8F1000T5E, symbol MY RESISTOR LIBRARY:0805W8F1000T5E
- added R506, R507: 47k, MY RESISTOR LIBRARY:0603WAF4702T5E, symbol MY RESISTOR LIBRARY:0603WAF4702T5E
- added U501: WM8978CGEFL_RV, MY AUDIO CODEC LIBRARY:WM8978CGEFL_RV_WQFN-32, symbol MY AUDIO CODEC LIBRARY:WM8978CGEFL_RV
Connections:
- net +3.3VA: now also C501.1, U501.31 (AVDD)
- net +3V3: now also C502.1, C503.1, R501.1, R502.1, U501.13 (DCVDD), U501.14 (DBVDD)
- net +5V: now also C504.1, U501.26 (SPKVDD)
- net AUXL: now also U501.19 (AUXL)
- net AUXR: now also U501.20 (AUXR)
- net GND: now also C501.2, C502.2, C503.2, C504.2, C505.2, J501.2, J502.2, R503.2, R506.2, R507.2, U501.12 (DGND), U501.24 (SPKGND), U501.28 (AGND), U501.33 (AGND)
- net IO0/MCLK: now also U501.11 (MCLK)
- net IO21/CODEC_SDIN: now also R501.2, U501.17 (SDIN)
- net IO22/CODEC_SCLK: now also R502.2, U501.16 (SCLK)
- net IO25/LRC: now also U501.7 (LRC)
- net IO26/DACDAT: now also U501.10 (DACDAT)
- net IO27/ADCDAT: now also U501.9 (ADCDAT)
- net IO33/BCLK: now also U501.8 (BCLK)
- net L2: now also U501.3 (L2/GPIO2)
- net LIN: now also U501.2 (LIN)
- net LIP: now also U501.1 (LIP)
- net LOUT1: now also U501.30 (LOUT1)
- net LOUT2: now also U501.25 (LOUT2)
- net MICBIAS: now also U501.32 (MICBIAS)
- net OUT3: now also U501.22 (OUT3)
- net OUT4: now also U501.21 (OUT4)
- net R2: now also U501.6 (R2/GPIO3)
- net RIN: now also U501.5 (RIN)
- net RIP: now also U501.4 (RIP)
- net ROUT1: now also U501.29 (ROUT1)
- net ROUT2: now also U501.23 (ROUT2)
- net VMID: now also C505.1, U501.27 (VMID)
- new net: J502.6, R504.1
- new net: C510.1, R504.2, R507.1
- new net: C508.2, J503.6
- new net: C511.1, R505.2, R506.1
- new net: J502.3, R505.1
- new net: C509.2, J503.3
- new net: C507.1, J501.3
- new net: C506.1, J501.6
- new net: R503.1, U501.18 (MODE)
- new net HP_L: C509.1
- new net HP_R: C508.1
- new net Line_In_L: C507.2
- new net Line_In_R: C506.2
- new net Line_Out_L: C511.2
- new net Line_Out_R: C510.2
- no-connect marks 1 -> 7
Other:
- note removed: "0R : for damping resistor value testing"

Commit message: updates
Parts:
- removed C506, C507: 1u, MY CAPACITOR LIBRARY:CL10A105KB8NNNC_0603, symbol MY CAPACITOR LIBRARY:CL10A105KB8NNNC
- removed J501: PJ-342B-TX-SMT, MY CONNECTOR LIBRARY:PJ-342B-TX-SMT, symbol MY CONNECTOR LIBRARY:PJ-342B-TX-SMT
Connections:
- net LOUT1 is gone; now on net HP_L: U501.30 (LOUT1)
- net OUT3 is gone; now on net Line_Out_L: U501.22 (OUT3)
- net OUT4 is gone; now on net Line_Out_R: U501.21 (OUT4)
- net ROUT1 is gone; now on net HP_R: U501.29 (ROUT1)
- net AUXL: no longer names the net of U501.19 (AUXL)
- net AUXR: no longer names the net of U501.20 (AUXR)
- net IO27/ADCDAT: no longer names the net of U501.9 (ADCDAT)
- net L2: no longer names the net of U501.3 (L2/GPIO2)
- net LIN: no longer names the net of U501.2 (LIN)
- net LIP: no longer names the net of U501.1 (LIP)
- net LOUT2: no longer names the net of U501.25 (LOUT2)
- net R2: no longer names the net of U501.6 (R2/GPIO3)
- net RIN: no longer names the net of U501.5 (RIN)
- net RIP: no longer names the net of U501.4 (RIP)
- net ROUT2: no longer names the net of U501.23 (ROUT2)
- no-connect marks 7 -> 15
Other:
- moved on the sheet: C508, C509, C510, C511, J502, J503, R504, R505, R506, R507

Commit message: updates
Connections:
- net GND: now also J503.2
- no-connect marks 15 -> 18
Other:
- note added: "AUDIO"
- note added: "LINE OUT & HEADPHONE"
- company: (none) -> Joël Ucedo
- title: (none) -> ESP32 SYNTH
- moved on the sheet: C501, C502, C503, C504, C505, C508, C509, C510, C511, J502, J503, R501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

Commit message: updates
Connections:
- net MICBIAS: no longer names the net of U501.32 (MICBIAS)
- no-connect marks 18 -> 19
Changed lines of the file:
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@@
   (no_connect (at 128.27 107.95))
   (no_connect (at 273.05 106.68))
+  (no_connect (at 168.91 106.68))
   (no_connect (at 273.05 104.14))
   (no_connect (at 128.27 140.97))
@@
     (stroke (width 0.5) (type default) (color 0 0 0 0))
   )
-  (wire (pts (xy 168.91 106.68) (xy 173.99 106.68))
-    (stroke (width 0) (type default) (color 0 0 0 0))
-  )
   (wire (pts (xy 274.32 165.1) (xy 276.86 165.1))
     (stroke (width 0) (type default) (color 0 0 0 0))
@@
     (effects (font (size 5 5) bold italic) (justify left bottom))
   )
-  (label "DACDAT" (at 119.38 110.49 0)
-    (effects (font (size 1.27 1.27) bold italic) (justify left bottom))
-  )
   (label "VMID" (at 171.45 102.87 0)
     (effects (font (size 1.27 1.27) bold italic) (justify left bottom))
@@
   (label "VMID" (at 152.4 213.36 0)
     (effects (font (size 1.27 1.27) bold italic) (justify left bottom))
-  )
-  (label "BCLK" (at 119.38 105.41 0)
-    (effects (font (size 1.27 1.27) (thickness 0.254) bold italic) (justify left bottom))
-  )
-  (label "MCLK" (at 119.38 113.03 0)
-    (effects (font (size 1.27 1.27) bold italic) (justify left bottom))
-  )
-  (label "LRC" (at 119.38 102.87 0)
-    (effects (font (size 1.27 1.27) (thickness 0.254) bold italic) (justify left bottom))
   )
   (global_label "HP_L" (shape input) (at 173.99 120.65 0) (fields_autoplaced)
@@
     )
   )
-  (global_label "MICBIAS" (shape input) (at 173.99 106.68 0) (fields_autoplaced)
-    (effects (font (size 1.27 1.27) bold italic) (justify left))
-    (property "Intersheet References" "${INTERSHEET_REFS}" (id 0) (at 184.3481 106.553 0)
-      (effects (font (size 1.27 1.27) bold italic) (justify left) hide)
-    )
-  )
   (global_label "IO0{slash}MCLK" (shape input) (at 102.87 113.03 180) (fields_autoplaced)
     (effects (font (size 1.27 1.27) (thickness 0.254) bold italic) (justify right))
@@
     (pin "2")
   )
-  (symbol (lib_id "MY RESISTOR LIBRARY:0805W8F1000T5E") (at 280.67 101.6 90) (unit 1)
-    (in_bom yes) (on_board yes)
-    (property "Reference" "R504" (id 0) (at 280.67 99.06 90))
-    (property "Value" "100R" (id 1) (at 280.67 104.14 90))
-    (property "Footprint" "MY RESISTOR LIBRARY:0805W8F1000T5E" (id 2) (at 280.67 103.378 90)
-      (effects (font (size 1.27 1.27)) hide)
-    )
-    (property "Datasheet" "~" (id 3) (at 280.67 101.6 0)
-      (effects (font (size 1.27 1.27)) hide)
-    )
-    (pin "1")
-    (pin "2")
-  )
   (symbol (lib_id "MY CAPACITOR LIBRARY:RVT1A221M0605") (at 288.29 154.94 270) (unit 1)
     (in_bom yes) (on_board yes)
@@
     (pin "1")
   )
-  (symbol (lib_id "MY RESISTOR LIBRARY:0603WAF4702T5E") (at 295.91 118.11 0) (unit 1)
-    (in_bom yes) (on_board yes) (fields_autoplaced)
-    (property "Reference" "R507" (id 0) (at 298.45 116.8399 0)
-      (effects (font (size 1.27 1.27)) (justify left))
-    )
-    (property "Value" "47k" (id 1) (at 298.45 119.3799 0)
-      (effects (font (size 1.27 1.27)) (justify left))
-    )
-    (property "Footprint" "MY RESISTOR LIBRARY:0603WAF4702T5E" (id 2) (at 294.132 118.11 90)
-      (effects (font (size 1.27 1.27)) hide)
-    )
-    (property "Datasheet" "~" (id 3) (at 295.91 118.11 0)
-      (effects (font (size 1.27 1.27)) hide)
-    )
-    (pin "1")
-    (pin "2")
-  )
   (symbol (lib_id "power:GND") (at 83.82 231.14 0) (unit 1)
     (in_bom yes) (on_board yes) (fields_autoplaced)
@@
     )
     (pin "1")
+  )
+  (symbol (lib_id "MY RESISTOR LIBRARY:0805W8F1000T5E") (at 280.67 109.22 90) (unit 1)
+    (in_bom yes) (on_board yes)
+    (property "Reference" "R505" (id 0) (at 280.67 106.68 90))
+    (property "Value" "100R" (id 1) (at 280.67 111.76 90))
+    (property "Footprint" "MY RESISTOR LIBRARY:0805W8F1000T5E" (id 2) (at 280.67 110.998 90)
+      (effects (font (size 1.27 1.27)) hide)
+    )
+    (property "Datasheet" "~" (id 3) (at 280.67 109.22 0)
+      (effects (font (size 1.27 1.27)) hide)
+    )
+    (pin "1")
+    (pin "2")
   )
   (symbol (lib_id "MY CAPACITOR LIBRARY:CL10A105KB8NNNC") (at 303.53 101.6 90) (unit 1)
@@
     )
     (property "Datasheet" "~" (id 3) (at 83.82 222.25 0)
-      (effects (font (size 1.27 1.27)) hide)
-    )
-    (pin "1")
-    (pin "2")
-  )
-  (symbol (lib_id "MY RESISTOR LIBRARY:0603WAF4702T5E") (at 289.56 118.11 0) (unit 1)
-    (in_bom yes) (on_board yes)
-    (property "Reference" "R506" (id 0) (at 281.94 116.84 0)
-      (effects (font (size 1.27 1.27)) (justify left))
-    )
-    (property "Value" "47k" (id 1) (at 283.21 119.38 0)
-      (effects (font (size 1.27 1.27)) (justify left))
-    )
-    (property "Footprint" "MY RESISTOR LIBRARY:0603WAF4702T5E" (id 2) (at 287.782 118.11 90)
-      (effects (font (size 1.27 1.27)) hide)
-    )
-    (property "Datasheet" "~" (id 3) (at 289.56 118.11 0)
       (effects (font (size 1.27 1.27)) hide)
     )
@@
     )
     (pin "1")
-  )
-  (symbol (lib_id "MY RESISTOR LIBRARY:0805W8F1000T5E") (at 280.67 109.22 90) (unit 1)
-    (in_bom yes) (on_board yes)
-    (property "Reference" "R505" (id 0) (at 280.67 106.68 90))
-    (property "Value" "100R" (id 1) (at 280.67 111.76 90))
-    (property "Footprint" "MY RESISTOR LIBRARY:0805W8F1000T5E" (id 2) (at 280.67 110.998 90)
-      (effects (font (size 1.27 1.27)) hide)
-    )
-    (property "Datasheet" "~" (id 3) (at 280.67 109.22 0)
-      (effects (font (size 1.27 1.27)) hide)
-    )
-    (pin "1")
-    (pin "2")
   )
   (symbol (lib_id "MY AUDIO CODEC LIBRARY:WM8978CGEFL_RV") (at 147.32 121.92 0) (unit 1)
@@
     (pin "1")
   )
+  (symbol (lib_id "MY RESISTOR LIBRARY:0603WAF4702T5E") (at 295.91 118.11 0) (unit 1)
+    (in_bom yes) (on_board yes)
+    (property "Reference" "R507" (id 0) (at 297.18 116.84 0)
+      (effects (font (size 1.27 1.27)) (justify left))
+    )
+    (property "Value" "47k" (id 1) (at 297.18 119.38 0)
+      (effects (font (size 1.27 1.27)) (justify left))
+    )
+    (property "Footprint" "MY RESISTOR LIBRARY:0603WAF4702T5E" (id 2) (at 294.132 118.11 90)
+      (effects (font (size 1.27 1.27)) hide)
+    )
+    (property "Datasheet" "~" (id 3) (at 295.91 118.11 0)
+      (effects (font (size 1.27 1.27)) hide)
+    )
+    (pin "1")
+    (pin "2")
+  )
+  (symbol (lib_id "MY RESISTOR LIBRARY:0603WAF4702T5E") (at 289.56 118.11 0) (unit 1)
+    (in_bom yes) (on_board yes)
+    (property "Reference" "R506" (id 0) (at 285.75 116.84 0)
+      (effects (font (size 1.27 1.27)) (justify left))
+    )
+    (property "Value" "47k" (id 1) (at 284.48 119.38 0)
+      (effects (font (size 1.27 1.27)) (justify left))
+    )
+    (property "Footprint" "MY RESISTOR LIBRARY:0603WAF4702T5E" (id 2) (at 287.782 118.11 90)
+      (effects (font (size 1.27 1.27)) hide)
+    )
+    (property "Datasheet" "~" (id 3) (at 289.56 118.11 0)
+      (effects (font (size 1.27 1.27)) hide)
+    )
+    (pin "1")
+    (pin "2")
+  )
   (symbol (lib_id "power:GND") (at 275.59 114.3 0) (unit 1)
     (in_bom yes) (on_board yes) (fields_autoplaced)
@@
     (pin "1")
   )
+  (symbol (lib_id "MY RESISTOR LIBRARY:0805W8F1000T5E") (at 280.67 101.6 90) (unit 1)
+    (in_bom yes) (on_board yes)
+    (property "Reference" "R504" (id 0) (at 280.67 99.06 90))
+    (property "Value" "100R" (id 1) (at 280.67 104.14 90))
+    (property "Footprint" "MY RESISTOR LIBRARY:0805W8F1000T5E" (id 2) (at 280.67 103.378 90)
+      (effects (font (size 1.27 1.27)) hide)
+    )
+    (property "Datasheet" "~" (id 3) (at 280.67 101.6 0)
+      (effects (font (size 1.27 1.27)) hide)
+    )
+    (pin "1")
+    (pin "2")
+  )
   (symbol (lib_id "MY RESISTOR LIBRARY:0603WAF1002T5E") (at 175.26 146.05 90) (unit 1)
