File: DESIGN FILES/audio.kicad_sch (KiCad schematic)
At the start: 19 parts, among them J502 PJ-342B-TX-SMT, J503 PJ-342B-TX-SMT, U501 WM8978CGEFL_RV

Commit message: updates
Parts:
- added C506, C507: 1u, MY CAPACITOR LIBRARY:CL10A105KB8NNNC_0603, symbol MY CAPACITOR LIBRARY:CL10A105KB8NNNC
- added J501: PJ-342B-TX-SMT, MY CONNECTOR LIBRARY:PJ-342B-TX-SMT, symbol MY CONNECTOR LIBRARY:PJ-342B-TX-SMT
Connections:
- net GND: now also J501.2
- net Line_in_L: now reaches U501.3 (L2/GPIO2)
- net Line_in_L: now also C507.2
- net Line_In_R: now reaches U501.6 (R2/GPIO3)
- net Line_In_R: now also C506.2
- net IO27/ADCDAT: now reaches U501.9 (ADCDAT)
- new net: C507.1, J501.3
- new net: C506.1, J501.6
Changed lines of the file:
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@@
   (junction (at 120.65 90.17) (diameter 0) (color 0 0 0 0)
   )
-  (no_connect (at 128.27 107.95))
+  (no_connect (at 274.32 199.39))
   (no_connect (at 273.05 106.68))
   (no_connect (at 168.91 106.68))
@@
   (no_connect (at 128.27 148.59))
   (no_connect (at 273.05 99.06))
-  (no_connect (at 128.27 125.73))
-  (no_connect (at 128.27 128.27))
+  (no_connect (at 274.32 204.47))
   (no_connect (at 168.91 125.73))
   (no_connect (at 168.91 128.27))
@@
   (no_connect (at 128.27 135.89))
   (no_connect (at 128.27 120.65))
+  (no_connect (at 274.32 207.01))
   (polyline (pts (xy 196.85 76.2) (xy 196.85 170.18))
     (stroke (width 0.5) (type default) (color 0 0 0 0))
@@
     (stroke (width 0) (type default) (color 0 0 0 0))
   )
-  (polyline (pts (xy 330.2 190.5) (xy 330.2 76.2))
+  (polyline (pts (xy 330.2 228.6) (xy 330.2 76.2))
     (stroke (width 0.5) (type default) (color 0 0 0 0))
   )
@@
     (stroke (width 0) (type default) (color 0 0 0 0))
   )
+  (wire (pts (xy 292.1 209.55) (xy 300.99 209.55))
+    (stroke (width 0) (type default) (color 0 0 0 0))
+  )
   (wire (pts (xy 168.91 139.7) (xy 173.99 139.7))
     (stroke (width 0) (type default) (color 0 0 0 0))
@@
     (stroke (width 0) (type default) (color 0 0 0 0))
   )
+  (wire (pts (xy 274.32 201.93) (xy 284.48 201.93))
+    (stroke (width 0) (type default) (color 0 0 0 0))
+  )
   (wire (pts (xy 152.4 213.36) (xy 152.4 218.44))
     (stroke (width 0) (type default) (color 0 0 0 0))
@@
     (stroke (width 0) (type default) (color 0 0 0 0))
   )
-  (polyline (pts (xy 241.3 190.5) (xy 330.2 190.5))
+  (polyline (pts (xy 241.3 228.6) (xy 330.2 228.6))
     (stroke (width 0.5) (type default) (color 0 0 0 0))
   )
@@
     (stroke (width 0) (type default) (color 0 0 0 0))
   )
+  (wire (pts (xy 292.1 201.93) (xy 300.99 201.93))
+    (stroke (width 0) (type default) (color 0 0 0 0))
+  )
   (wire (pts (xy 168.91 137.16) (xy 173.99 137.16))
     (stroke (width 0) (type default) (color 0 0 0 0))
   )
+  (wire (pts (xy 274.32 209.55) (xy 284.48 209.55))
+    (stroke (width 0) (type default) (color 0 0 0 0))
+  )
   (wire (pts (xy 134.62 226.06) (xy 134.62 231.14))
     (stroke (width 0) (type default) (color 0 0 0 0))
@@
     (stroke (width 0) (type default) (color 0 0 0 0))
   )
+  (wire (pts (xy 276.86 212.09) (xy 276.86 214.63))
+    (stroke (width 0) (type default) (color 0 0 0 0))
+  )
+  (wire (pts (xy 274.32 212.09) (xy 276.86 212.09))
+    (stroke (width 0) (type default) (color 0 0 0 0))
+  )
   (wire (pts (xy 168.91 92.71) (xy 171.45 92.71))
     (stroke (width 0) (type default) (color 0 0 0 0))
@@
     (stroke (width 0) (type default) (color 0 0 0 0))
   )
+  (wire (pts (xy 102.87 107.95) (xy 128.27 107.95))
+    (stroke (width 0) (type default) (color 0 0 0 0))
+  )
+  (wire (pts (xy 123.19 128.27) (xy 128.27 128.27))
+    (stroke (width 0) (type default) (color 0 0 0 0))
+  )
   (wire (pts (xy 307.34 101.6) (xy 309.88 101.6))
     (stroke (width 0) (type default) (color 0 0 0 0))
@@
     (stroke (width 0) (type default) (color 0 0 0 0))
   )
+  (wire (pts (xy 123.19 125.73) (xy 128.27 125.73))
+    (stroke (width 0) (type default) (color 0 0 0 0))
+  )
   (wire (pts (xy 295.91 101.6) (xy 299.72 101.6))
     (stroke (width 0) (type default) (color 0 0 0 0))
   )
-  (polyline (pts (xy 241.3 76.2) (xy 241.3 190.5))
+  (polyline (pts (xy 241.3 76.2) (xy 241.3 228.6))
     (stroke (width 0.5) (type default) (color 0 0 0 0))
   )
@@
   (label "VMID" (at 152.4 213.36 0)
     (effects (font (size 1.27 1.27) bold italic) (justify left bottom))
+  )
+  (global_label "Line_in_L" (shape input) (at 300.99 209.55 0) (fields_autoplaced)
+    (effects (font (size 1.27 1.27) bold italic) (justify left))
+    (property "Intersheet References" "${INTERSHEET_REFS}" (id 0) (at 312.4367 209.423 0)
+      (effects (font (size 1.27 1.27) bold italic) (justify left) hide)
+    )
+  )
+  (global_label "Line_In_R" (shape input) (at 300.99 201.93 0) (fields_autoplaced)
+    (effects (font (size 1.27 1.27) bold italic) (justify left))
+    (property "Intersheet References" "${INTERSHEET_REFS}" (id 0) (at 312.6786 201.803 0)
+      (effects (font (size 1.27 1.27) bold italic) (justify left) hide)
+    )
+  )
+  (global_label "Line_in_L" (shape input) (at 123.19 128.27 180) (fields_autoplaced)
+    (effects (font (size 1.27 1.27) bold italic) (justify right))
+    (property "Intersheet References" "${INTERSHEET_REFS}" (id 0) (at 111.7433 128.397 0)
+      (effects (font (size 1.27 1.27) bold italic) (justify right) hide)
+    )
   )
   (global_label "HP_L" (shape input) (at 173.99 120.65 0) (fields_autoplaced)
@@
     )
   )
+  (global_label "Line_In_R" (shape input) (at 123.19 125.73 180) (fields_autoplaced)
+    (effects (font (size 1.27 1.27) bold italic) (justify right))
+    (property "Intersheet References" "${INTERSHEET_REFS}" (id 0) (at 111.5014 125.857 0)
+      (effects (font (size 1.27 1.27) bold italic) (justify right) hide)
+    )
+  )
   (global_label "Line_Out_L" (shape input) (at 173.99 137.16 0) (fields_autoplaced)
     (effects (font (size 1.27 1.27) bold italic) (justify left))
@@
     )
   )
+  (global_label "IO27{slash}ADCDAT" (shape input) (at 102.87 107.95 180) (fields_autoplaced)
+    (effects (font (size 1.27 1.27) (thickness 0.254) bold italic) (justify right))
+    (property "Intersheet References" "${INTERSHEET_REFS}" (id 0) (at 87.3714 108.077 0)
+      (effects (font (size 1.27 1.27) (thickness 0.254) bold italic) (justify right) hide)
+    )
+  )
   (global_label "HP_R" (shape input) (at 300.99 154.94 0) (fields_autoplaced)
     (effects (font (size 1.27 1.27) bold italic) (justify left))
@@
     )
     (pin "1")
+  )
+  (symbol (lib_id "MY CAPACITOR LIBRARY:CL10A105KB8NNNC") (at 288.29 209.55 90) (unit 1)
+    (in_bom yes) (on_board yes)
+    (property "Reference" "C507" (id 0) (at 284.48 207.01 90))
+    (property "Value" "1u" (id 1) (at 292.1 207.01 90))
+    (property "Footprint" "MY CAPACITOR LIBRARY:CL10A105KB8NNNC_0603" (id 2) (at 292.1 208.5848 0)
+      (effects (font (size 1.27 1.27)) hide)
+    )
+    (property "Datasheet" "~" (id 3) (at 288.29 209.55 0)
+      (effects (font (size 1.27 1.27)) hide)
+    )
+    (pin "1")
+    (pin "2")
   )
   (symbol (lib_id "power:GND") (at 83.82 231.14 0) (unit 1)
@@
     (pin "1")
     (pin "2")
+  )
+  (symbol (lib_name "PJ-342B-TX-SMT_1") (lib_id "MY CONNECTOR LIBRARY:PJ-342B-TX-SMT") (at 260.35 205.74 0) (unit 1)
+    (in_bom yes) (on_board yes) (fields_autoplaced)
+    (property "Reference" "J501" (id 0) (at 259.715 193.04 0)
+      (effects (font (size 1.524 1.524)))
+    )
+    (property "Value" "PJ-342B-TX-SMT" (id 1) (at 259.715 196.85 0)
+      (effects (font (size 1.524 1.524)))
+    )
+    (property "Footprint" "MY CONNECTOR LIBRARY:PJ-342B-TX-SMT" (id 2) (at 255.27 195.58 0)
+      (effects (font (size 1.524 1.524)) hide)
+    )
+    (property "Datasheet" "" (id 3) (at 274.32 199.39 0)
+      (effects (font (size 1.524 1.524)))
+    )
+    (pin "2")
+    (pin "3")
+    (pin "4")
+    (pin "5")
+    (pin "6")
+    (pin "7")
   )
   (symbol (lib_id "MY CAPACITOR LIBRARY:CL10A475KO8NNNC") (at 115.57 222.25 0) (unit 1)
@@
     (pin "1")
   )
+  (symbol (lib_id "MY CAPACITOR LIBRARY:CL10A105KB8NNNC") (at 288.29 201.93 90) (unit 1)
+    (in_bom yes) (on_board yes)
+    (property "Reference" "C506" (id 0) (at 284.48 199.39 90))
+    (property "Value" "1u" (id 1) (at 292.1 199.39 90))
+    (property "Footprint" "MY CAPACITOR LIBRARY:CL10A105KB8NNNC_0603" (id 2) (at 292.1 200.9648 0)
+      (effects (font (size 1.27 1.27)) hide)
+    )
+    (property "Datasheet" "~" (id 3) (at 288.29 201.93 0)
+      (effects (font (size 1.27 1.27)) hide)
+    )
+    (pin "1")
+    (pin "2")
+  )
   (symbol (lib_id "power:+3V3") (at 115.57 213.36 0) (unit 1)
     (in_bom yes) (on_board yes) (fields_autoplaced)
@@
     (pin "2")
   )
+  (symbol (lib_id "power:GND") (at 276.86 214.63 0) (unit 1)
+    (in_bom yes) (on_board yes) (fields_autoplaced)
+    (property "Reference" "#PWR0501" (id 0) (at 276.86 220.98 0)
+      (effects (font (size 1.27 1.27)) hide)
+    )
+    (property "Value" "GND" (id 1) (at 276.86 219.71 0))
+    (property "Footprint" "" (id 2) (at 276.86 214.63 0)
+      (effects (font (size 1.27 1.27)) hide)
+    )
+    (property "Datasheet" "" (id 3) (at 276.86 214.63 0)
+      (effects (font (size 1.27 1.27)) hide)
+    )
+    (pin "1")
+  )
   (symbol (lib_id "MY RESISTOR LIBRARY:0603WAF1002T5E") (at 175.26 146.05 90) (unit 1)
