File: DESIGN FILES/audio.kicad_sch (KiCad schematic)
At the start: 22 parts, among them J501 PJ-342B-TX-SMT, J502 PJ-342B-TX-SMT, J503 PJ-342B-TX-SMT, U501 WM8978CGEFL_RV

Commit message: updates
Other:
- note added: "LINE IN/OUT & HEADPHONE"
- note removed: "LINE OUT & HEADPHONE"
- moved on the sheet: C506, C507, C508, C509, C510, C511, J501, J502, J503, R504, R505, R506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

Commit message: updates
Parts:
- removed R504, R505: 100R, MY RESISTOR LIBRARY:0805W8F1000T5E, symbol MY RESISTOR LIBRARY:0805W8F1000T5E
- added R504, R505: 100R, MY RESISTOR LIBRARY:0603WAF1000T5E, symbol MY RESISTOR LIBRARY:0603WAF1000T5E
Connections:
- net at J502.3: now also R505.1
- net at C511.1, R506.1: now also R505.2
- net at C510.1, R507.1: now also R504.2
- net at J502.6: now also R504.1
Changed lines of the file:
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@@
+    (pin "2")
+  )
+  (symbol (lib_id "MY RESISTOR LIBRARY:0603WAF1000T5E") (at 297.18 107.95 90) (unit 1)
+    (in_bom yes) (on_board yes)
+    (property "Reference" "R505" (id 0) (at 297.18 105.41 90))
+    (property "Value" "100R" (id 1) (at 297.18 110.49 90))
+    (property "Footprint" "MY RESISTOR LIBRARY:0603WAF1000T5E" (id 2) (at 297.18 109.728 90)
+      (effects (font (size 1.27 1.27)) hide)
+    )
+    (property "Datasheet" "~" (id 3) (at 297.18 107.95 0)
+      (effects (font (size 1.27 1.27)) hide)
+    )
+    (pin "1")
     (pin "2")
   )
@@
     )
     (pin "1")
-  )
-  (symbol (lib_id "MY RESISTOR LIBRARY:0805W8F1000T5E") (at 297.18 107.95 90) (unit 1)
-    (in_bom yes) (on_board yes)
-    (property "Reference" "R505" (id 0) (at 297.18 105.41 90))
-    (property "Value" "100R" (id 1) (at 297.18 110.49 90))
-    (property "Footprint" "MY RESISTOR LIBRARY:0805W8F1000T5E" (id 2) (at 297.18 109.728 90)
-      (effects (font (size 1.27 1.27)) hide)
-    )
-    (property "Datasheet" "~" (id 3) (at 297.18 107.95 0)
-      (effects (font (size 1.27 1.27)) hide)
-    )
-    (pin "1")
-    (pin "2")
   )
   (symbol (lib_id "MY CAPACITOR LIBRARY:CL10A105KB8NNNC") (at 320.04 100.33 90) (unit 1)
@@
     (pin "1")
   )
+  (symbol (lib_id "MY RESISTOR LIBRARY:0603WAF1000T5E") (at 297.18 100.33 90) (unit 1)
+    (in_bom yes) (on_board yes)
+    (property "Reference" "R504" (id 0) (at 297.18 97.79 90))
+    (property "Value" "100R" (id 1) (at 297.18 102.87 90))
+    (property "Footprint" "MY RESISTOR LIBRARY:0603WAF1000T5E" (id 2) (at 297.18 102.108 90)
+      (effects (font (size 1.27 1.27)) hide)
+    )
+    (property "Datasheet" "~" (id 3) (at 297.18 100.33 0)
+      (effects (font (size 1.27 1.27)) hide)
+    )
+    (pin "1")
+    (pin "2")
+  )
   (symbol (lib_id "power:GND") (at 306.07 123.19 0) (unit 1)
     (in_bom yes) (on_board yes) (fields_autoplaced)
@@
   (symbol (lib_id "MY RESISTOR LIBRARY:0603WAF4702T5E") (at 306.07 116.84 0) (unit 1)
     (in_bom yes) (on_board yes)
-    (property "Reference" "R506" (id 0) (at 302.26 115.57 0)
+    (property "Reference" "R506" (id 0) (at 299.72 115.57 0)
       (effects (font (size 1.27 1.27)) (justify left))
     )
@@
     (pin "1")
   )
-  (symbol (lib_id "MY RESISTOR LIBRARY:0805W8F1000T5E") (at 297.18 100.33 90) (unit 1)
-    (in_bom yes) (on_board yes)
-    (property "Reference" "R504" (id 0) (at 297.18 97.79 90))
-    (property "Value" "100R" (id 1) (at 297.18 102.87 90))
-    (property "Footprint" "MY RESISTOR LIBRARY:0805W8F1000T5E" (id 2) (at 297.18 102.108 90)
-      (effects (font (size 1.27 1.27)) hide)
-    )
-    (property "Datasheet" "~" (id 3) (at 297.18 100.33 0)
-      (effects (font (size 1.27 1.27)) hide)
-    )
-    (pin "1")
-    (pin "2")
-  )
   (symbol (lib_id "power:GND") (at 293.37 213.36 0) (unit 1)
