File: DESIGN FILES/midi.kicad_sch (KiCad schematic)
At the start: 0 parts

Commit message: updates
Parts:
- added C? (x2): 100nF, soundsom:CC0603KRX7R9BB104_0603, symbol soundsom:CC0603KRX7R9BB104
- added D?: 1N4148W, soundsom:1N4148W_SOD-123, symbol soundsom:1N4148W
- added R?: 220R, soundsom:0603WAF2200T5E_0603, symbol soundsom:0603WAF2200T5E
- added R?: 10k, soundsom:0603WAF1002T5E_0603, symbol soundsom:0603WAF1002T5E
- added U?: 6N137S1(TA), soundsom:6N137S1_TA_SMD-8P, symbol soundsom:6N137S1(TA)
- added U?: 74HC04D,653, soundsom:74HC04D_653_SOIC-14, symbol soundsom:74HC04D,653
Connections:
- new net: D?.1 (K), R?.1, U?.2 (A)
- new net: U?.11 (5A), U?.12 (6Y)
- new net: U?.2 (1Y), U?.3 (2A)
- new net +3V3: C?.1, R?.1, U?.14 (VCC)
- new net +5V: C?.1, U?.8 (VCC)
- new net GND: C?.2, C?.2, U?.5 (GND), U?.7 (GND)
- new net MIDI_IN: R?.2, U?.1 (1A), U?.6 (VO)
- new net MIDI_IN_RING: R?.2
- new net MIDI_IN_TIP: D?.2 (A), U?.3 (K)
- new net MIDI_OUT: U?.13 (6A)
- new net OUT: U?.10 (5Y)
- new net THRU: U?.4 (2Y)
- no-connect marks 0 -> 5
Other:
- note added: "MIDI IN"
- note added: "MIDI OUT & THRU"

Commit message: updates
Parts:
- removed C? (x2): 100nF, soundsom:CC0603KRX7R9BB104_0603, symbol soundsom:CC0603KRX7R9BB104
- removed D?: 1N4148W, soundsom:1N4148W_SOD-123, symbol soundsom:1N4148W
- removed R?: 220R, soundsom:0603WAF2200T5E_0603, symbol soundsom:0603WAF2200T5E
- removed R?: 10k, soundsom:0603WAF1002T5E_0603, symbol soundsom:0603WAF1002T5E
- removed U?: 6N137S1(TA), soundsom:6N137S1_TA_SMD-8P, symbol soundsom:6N137S1(TA)
- removed U?: 74HC04D,653, soundsom:74HC04D_653_SOIC-14, symbol soundsom:74HC04D,653
- added C601, C602: 100n, MY CAPACITOR LIBRARY:CC0603KRX7R9BB104_0603, symbol MY CAPACITOR LIBRARY:CC0603KRX7R9BB104
- added D601: 1N4148W, MY DIODE LIBRARY:1N4148W_SOD-123, symbol MY DIODE LIBRARY:1N4148W
- added J601, J602, J603: PJ-342B-TX-SMT, MY CONNECTOR LIBRARY:PJ-342B-TX-SMT, symbol MY CONNECTOR LIBRARY:PJ-342B-TX-SMT
- added R601: 220R, MY RESISTOR LIBRARY:0603WAF2200T5E, symbol MY RESISTOR LIBRARY:0603WAF2200T5E
- added R602: 10k, MY RESISTOR LIBRARY:0603WAF1002T5E, symbol MY RESISTOR LIBRARY:0603WAF1002T5E
- added R603, R604, R605, R606: 33R, MY RESISTOR LIBRARY:0805W8F330JT5E, symbol MY RESISTOR LIBRARY:0603WAF330JT5E
- added U601: 6N137S1(TA), MY OPTO IC LIBRARY:6N137S1_TA_SMD-8P, symbol MY OPTO IC LIBRARY:6N137S1(TA)
- added U602: 74HC04D,653, MY IC LIBRARY:74HC04D_653_SOIC-14, symbol MY IC LIBRARY:74HC04D,653
Connections:
- net +3V3: now also C602.1, R602.1, R603.2, R605.2, U602.14 (VCC)
- net +5V: now also C601.1, U601.8 (VCC)
- net GND: now also C601.2, C602.2, J602.2, J603.2, U601.5 (GND), U602.7 (GND)
- net MIDI_IN: now also R602.2, U601.6 (VO), U602.1 (1A)
- net MIDI_IN_RING: now also J601.6, R601.2
- net MIDI_IN_TIP: now also D601.2 (A), J601.3, U601.3 (K)
- net MIDI_OUT: now also U602.13 (6A)
- net OUT: now also R604.2, U602.10 (5Y)
- net THRU: now also R606.2, U602.4 (2Y)
- new net: J603.3, R606.1
- new net: J603.6, R605.1
- new net: D601.1 (K), R601.1, U601.2 (A)
- new net: U602.11 (5A), U602.12 (6Y)
- new net: U602.2 (1Y), U602.3 (2A)
- new net: J602.6, R603.1
- new net: J602.3, R604.1
- no-connect marks 5 -> 15

Commit message: updates
Parts:
- removed J603: PJ-342B-TX-SMT, MY CONNECTOR LIBRARY:PJ-342B-TX-SMT, symbol MY CONNECTOR LIBRARY:PJ-342B-TX-SMT
- removed R605, R606: 33R, MY RESISTOR LIBRARY:0805W8F330JT5E, symbol MY RESISTOR LIBRARY:0603WAF330JT5E
Connections:
- net THRU is gone; now on net OUT: U602.4 (2Y)
- net MIDI_IN: no longer U602.1 (1A)
- net MIDI_OUT: now also U602.1 (1A); no longer U602.13 (6A)
- net OUT: no longer U602.10 (5Y)
- net at U602.11 (5A): no longer U602.12 (6Y)
- net at U602.2 (1Y): no longer U602.3 (2A)
- no-connect marks 15 -> 18
Other:
- moved on the sheet: C602, J601, J602, R603, R604

Commit message: updates
Connections:
- net at U602.2 (1Y): now also U602.3 (2A)
- no-connect marks 18 -> 16
Other:
- note added: "MIDI"
- company: (none) -> Joël Ucedo
- title: (none) -> ESP32 SYNTH
- moved on the sheet: C601, C602, D601, J601, J602, R601, R602, R603, R604, U601, U602

Commit message: updates
Parts:
- R603, R604: footprint MY RESISTOR LIBRARY:0805W8F330JT5E -> MY RESISTOR LIBRARY:0603WAF330JT5E
Changed lines of the file:
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@@
     )
+  )
+  (symbol (lib_id "MY RESISTOR LIBRARY:0603WAF330JT5E") (at 309.88 180.34 90) (unit 1)
+    (in_bom yes) (on_board yes)
+    (property "Reference" "R604" (id 0) (at 309.88 177.8 90))
+    (property "Value" "33R" (id 1) (at 309.88 182.88 90))
+    (property "Footprint" "MY RESISTOR LIBRARY:0603WAF330JT5E" (id 2) (at 309.88 182.118 90)
+      (effects (font (size 1.27 1.27)) hide)
+    )
+    (property "Datasheet" "~" (id 3) (at 309.88 180.34 0)
+      (effects (font (size 1.27 1.27)) hide)
+    )
+    (pin "1")
+    (pin "2")
   )
   (symbol (lib_id "MY OPTO IC LIBRARY:6N137S1(TA)") (at 148.59 109.22 0) (unit 1)
@@
     (pin "9")
   )
+  (symbol (lib_name "PJ-342B-TX-SMT_1") (lib_id "MY CONNECTOR LIBRARY:PJ-342B-TX-SMT") (at 144.78 179.07 0) (unit 1)
+    (in_bom yes) (on_board yes) (fields_autoplaced)
+    (property "Reference" "J601" (id 0) (at 144.145 166.37 0)
+      (effects (font (size 1.524 1.524)))
+    )
+    (property "Value" "PJ-342B-TX-SMT" (id 1) (at 144.145 170.18 0)
+      (effects (font (size 1.524 1.524)))
+    )
+    (property "Footprint" "MY CONNECTOR LIBRARY:PJ-342B-TX-SMT" (id 2) (at 139.7 168.91 0)
+      (effects (font (size 1.524 1.524)) hide)
+    )
+    (property "Datasheet" "" (id 3) (at 158.75 172.72 0)
+      (effects (font (size 1.524 1.524)))
+    )
+    (pin "2")
+    (pin "3")
+    (pin "4")
+    (pin "5")
+    (pin "6")
+    (pin "7")
+  )
+  (symbol (lib_name "PJ-342B-TX-SMT_1") (lib_id "MY CONNECTOR LIBRARY:PJ-342B-TX-SMT") (at 285.75 176.53 0) (unit 1)
+    (in_bom yes) (on_board yes) (fields_autoplaced)
+    (property "Reference" "J602" (id 0) (at 285.115 163.83 0)
+      (effects (font (size 1.524 1.524)))
+    )
+    (property "Value" "PJ-342B-TX-SMT" (id 1) (at 285.115 167.64 0)
+      (effects (font (size 1.524 1.524)))
+    )
+    (property "Footprint" "MY CONNECTOR LIBRARY:PJ-342B-TX-SMT" (id 2) (at 280.67 166.37 0)
+      (effects (font (size 1.524 1.524)) hide)
+    )
+    (property "Datasheet" "" (id 3) (at 299.72 170.18 0)
+      (effects (font (size 1.524 1.524)))
+    )
+    (pin "2")
+    (pin "3")
+    (pin "4")
+    (pin "5")
+    (pin "6")
+    (pin "7")
+  )
+  (symbol (lib_id "power:+3V3") (at 176.53 85.09 0) (unit 1)
+    (in_bom yes) (on_board yes) (fields_autoplaced)
+    (property "Reference" "#PWR0151" (id 0) (at 176.53 88.9 0)
+      (effects (font (size 1.27 1.27)) hide)
+    )
+    (property "Value" "+3V3" (id 1) (at 176.53 80.01 0))
+    (property "Footprint" "" (id 2) (at 176.53 85.09 0)
+      (effects (font (size 1.27 1.27)) hide)
+    )
+    (property "Datasheet" "" (id 3) (at 176.53 85.09 0)
+      (effects (font (size 1.27 1.27)) hide)
+    )
+    (pin "1")
+  )
   (symbol (lib_id "MY RESISTOR LIBRARY:0603WAF330JT5E") (at 309.88 172.72 90) (unit 1)
     (in_bom yes) (on_board yes)
     (property "Reference" "R603" (id 0) (at 309.88 170.18 90))
     (property "Value" "33R" (id 1) (at 309.88 175.26 90))
-    (property "Footprint" "MY RESISTOR LIBRARY:0805W8F330JT5E" (id 2) (at 309.88 174.498 90)
+    (property "Footprint" "MY RESISTOR LIBRARY:0603WAF330JT5E" (id 2) (at 309.88 174.498 90)
       (effects (font (size 1.27 1.27)) hide)
     )
@@
     (pin "1")
     (pin "2")
-  )
-  (symbol (lib_name "PJ-342B-TX-SMT_1") (lib_id "MY CONNECTOR LIBRARY:PJ-342B-TX-SMT") (at 144.78 179.07 0) (unit 1)
-    (in_bom yes) (on_board yes) (fields_autoplaced)
-    (property "Reference" "J601" (id 0) (at 144.145 166.37 0)
-      (effects (font (size 1.524 1.524)))
-    )
-    (property "Value" "PJ-342B-TX-SMT" (id 1) (at 144.145 170.18 0)
-      (effects (font (size 1.524 1.524)))
-    )
-    (property "Footprint" "MY CONNECTOR LIBRARY:PJ-342B-TX-SMT" (id 2) (at 139.7 168.91 0)
-      (effects (font (size 1.524 1.524)) hide)
-    )
-    (property "Datasheet" "" (id 3) (at 158.75 172.72 0)
-      (effects (font (size 1.524 1.524)))
-    )
-    (pin "2")
-    (pin "3")
-    (pin "4")
-    (pin "5")
-    (pin "6")
-    (pin "7")
-  )
-  (symbol (lib_name "PJ-342B-TX-SMT_1") (lib_id "MY CONNECTOR LIBRARY:PJ-342B-TX-SMT") (at 285.75 176.53 0) (unit 1)
-    (in_bom yes) (on_board yes) (fields_autoplaced)
-    (property "Reference" "J602" (id 0) (at 285.115 163.83 0)
-      (effects (font (size 1.524 1.524)))
-    )
-    (property "Value" "PJ-342B-TX-SMT" (id 1) (at 285.115 167.64 0)
-      (effects (font (size 1.524 1.524)))
-    )
-    (property "Footprint" "MY CONNECTOR LIBRARY:PJ-342B-TX-SMT" (id 2) (at 280.67 166.37 0)
-      (effects (font (size 1.524 1.524)) hide)
-    )
-    (property "Datasheet" "" (id 3) (at 299.72 170.18 0)
-      (effects (font (size 1.524 1.524)))
-    )
-    (pin "2")
-    (pin "3")
-    (pin "4")
-    (pin "5")
-    (pin "6")
-    (pin "7")
-  )
-  (symbol (lib_id "power:+3V3") (at 176.53 85.09 0) (unit 1)
-    (in_bom yes) (on_board yes) (fields_autoplaced)
-    (property "Reference" "#PWR0151" (id 0) (at 176.53 88.9 0)
-      (effects (font (size 1.27 1.27)) hide)
-    )
-    (property "Value" "+3V3" (id 1) (at 176.53 80.01 0))
-    (property "Footprint" "" (id 2) (at 176.53 85.09 0)
-      (effects (font (size 1.27 1.27)) hide)
-    )
-    (property "Datasheet" "" (id 3) (at 176.53 85.09 0)
-      (effects (font (size 1.27 1.27)) hide)
-    )
-    (pin "1")
   )
   (symbol (lib_id "power:GND") (at 160.02 118.11 0) (unit 1)
@@
     (pin "1")
   )
-  (symbol (lib_id "MY RESISTOR LIBRARY:0603WAF330JT5E") (at 309.88 180.34 90) (unit 1)
-    (in_bom yes) (on_board yes)
-    (property "Reference" "R604" (id 0) (at 309.88 177.8 90))
-    (property "Value" "33R" (id 1) (at 309.88 182.88 90))
-    (property "Footprint" "MY RESISTOR LIBRARY:0805W8F330JT5E" (id 2) (at 309.88 182.118 90)
-      (effects (font (size 1.27 1.27)) hide)
-    )
-    (property "Datasheet" "~" (id 3) (at 309.88 180.34 0)
-      (effects (font (size 1.27 1.27)) hide)
-    )
-    (pin "1")
-    (pin "2")
-  )
   (symbol (lib_id "power:GND") (at 166.37 100.33 0) (unit 1)

Commit message: updates
Parts:
- added J603: PJ-342B-TX-SMT, MY CONNECTOR LIBRARY:PJ-342B-TX-SMT, symbol MY CONNECTOR LIBRARY:PJ-342B-TX-SMT
- added R605, R606: 33R, MY RESISTOR LIBRARY:0603WAF330JT5E, symbol MY RESISTOR LIBRARY:0603WAF330JT5E
Connections:
- net +3V3: now also R605.2
- net GND: now also J603.2
- net MIDI_IN: now also U602.13 (6A)
- net THRU: now reaches U602.10 (5Y)
- net THRU: now also R606.2
- net at U602.11 (5A): now also U602.12 (6Y)
- new net: J603.3, R606.1
- new net: J603.6, R605.1
- no-connect marks 16 -> 15
Other:
- moved on the sheet: C602, J602, R603, R604
