File: DESIGN FILES/midi.kicad_sch (KiCad schematic)
At the start: 14 parts, among them J601 PJ-342B-TX-SMT, J602 PJ-342B-TX-SMT, J603 PJ-342B-TX-SMT, U601 6N137S1(TA), U602 74HC04D,653

Commit message: updates
Changed lines of the file:
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@@
   )
   (symbol (lib_id "MY DIODE LIBRARY:1N4148W") (at 133.35 111.76 0) (unit 1)
-    (in_bom yes) (on_board yes) (fields_autoplaced)
-    (property "Reference" "D601" (id 0) (at 133.35 105.41 0))
-    (property "Value" "1N4148W" (id 1) (at 133.35 107.95 0))
+    (in_bom yes) (on_board yes)
+    (property "Reference" "D601" (id 0) (at 133.35 109.22 0))
+    (property "Value" "1N4148W" (id 1) (at 133.35 114.3 0))
     (property "Footprint" "MY DIODE LIBRARY:1N4148W_SOD-123" (id 2) (at 133.35 116.205 0)
       (effects (font (size 1.27 1.27)) hide)
