File: DESIGN FILES/ESP32 synth.kicad_pcb (KiCad board)
At the start: 2 copper layers, 127 x 127 mm, 108 parts, among them J401 YTC-TC16S-28, J402 JTAG, J501 PJ-342B-TX-SMT, J502 PJ-342B-TX-SMT, J503 PJ-342B-TX-SMT, J601 PJ-342B-TX-SMT, J602 PJ-342B-TX-SMT, J603 PJ-342B-TX-SMT, J801 TF-15x15, J802 TFT-LCD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

Commit message: updates
Parts:
- moved C401 274.4 mm to (401.4, 45.1)
- moved C402 274.4 mm to (401.4, 40.1)
- moved C404 274.4 mm to (389.4, 59.2)
- moved C406 274.4 mm to (405.4, 42.6)
- moved D402 274.4 mm to (380.5, 60.5)
- moved R401 274.4 mm to (401.4, 42.6)
- moved R407 274.4 mm to (405.4, 45.1)
- moved Q401 258.8 mm to (104.9, 54.5)
- moved U401 258.8 mm to (135.1, 50.8)
- moved C407 258.8 mm to (129.5, 23.6)
- moved C501 258.8 mm to (102.4, 69.8)
- moved C502 258.8 mm to (102.4, 67.3)
- moved C505 258.8 mm to (106.4, 69.8)
- moved J401 258.8 mm to (196.1, 62.5)
- moved J801 258.8 mm to (80.9, 62.5)
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
Commit message: updates
Parts:
- moved J802 418.9 mm to (74.7, 51.8)
- moved H104 378.6 mm to (75.2, 158.0)
- moved C510 366.8 mm to (95.8, 44.7), turned to -90 degrees
- moved H101 364.6 mm to (75.2, 37.6)
- moved R507 356.4 mm to (96.5, 42.2)
- moved J402 356.4 mm to (135.6, 155.7)
- moved C509 352.3 mm to (102.4, 56.1), turned to 90 degrees
- moved C511 342.9 mm to (109.7, 48.5)
- moved C508 336.0 mm to (92.7, 56.1), turned to 90 degrees
- moved R504 333.5 mm to (96.0, 39.4), turned to -90 degrees
- moved C506 329.7 mm to (109.2, 39.6), turned to -90 degrees
- moved J503 329.0 mm to (88.9, 39.3)
- moved R505 328.9 mm to (109.0, 43.4), turned to -90 degrees
- moved J501 325.4 mm to (115.8, 39.4)
- moved R506 322.7 mm to (109.7, 46.5)
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Routing:
- net USB_D+: track 0.00 -> 27.4 mm
- net USB_D-: track 0.00 -> 25.0 mm
- net /MCU - USB - JTAG/DTR: track 0.00 -> 11.9 mm
- net /MCU - USB - JTAG/RTS: track 0.00 -> 7.78 mm
- net Net-(J401-PadB5): track 0.00 -> 5.67 mm
- net Net-(J401-PadA5): track 0.00 -> 5.14 mm
- net Net-(Q401-Pad1): track 0.00 -> 3.03 mm
- net Net-(Q402-Pad1): track 0.00 -> 2.52 mm
Other:
- outline, holes or cut-outs redrawn

Commit message: updates
Parts:
- removed C506, C507: 1u, MY CAPACITOR LIBRARY:CL10A105KB8NNNC_0603
- removed C801: 22u, MY CAPACITOR LIBRARY:0603_CL10A226MQ8NRNC
- removed FB801: 600R, MY FERRITE BEAD LIBRARY:UPZ1608U601-1R3TF_0603
- removed J402: JTAG, MY CONNECTOR LIBRARY:PZ127VS-12-10-H10-A38
- removed J501, J603: PJ-342B-TX-SMT, MY CONNECTOR LIBRARY:PJ-342B-TX-SMT
- removed J801: TF-15x15, MY CONNECTOR LIBRARY:TF-15x15_smd
- removed J802: TFT-LCD, MY CONNECTOR LIBRARY:801-87-008-10-003101
- removed R605, R606: 33R, MY RESISTOR LIBRARY:0805W8F330JT5E
- removed R801, R802, R803, R804, R805: 47k, MY RESISTOR LIBRARY:0603WAF4702T5E
- removed U702: ENCODER, MY ENCODER LIBRARY:ENC_PEC12R-4025F-S0024
Connections:
- net /MCU - USB - JTAG/DTR renamed /MCU - USB/DTR
- net /MCU - USB - JTAG/EN renamed /MCU - USB/EN
- net /MCU - USB - JTAG/RTS renamed /MCU - USB/RTS
- RV701 pad 1: unconnected-(RV701-Pad1) -> GND
- RV701 pad 2: unconnected-(RV701-Pad2) -> MUX_IO6
- RV701 pad 3: unconnected-(RV701-Pad3) -> +3V3
- RV702 pad 1: unconnected-(RV702-Pad1) -> GND
- RV702 pad 2: unconnected-(RV702-Pad2) -> MUX_IO4
- RV702 pad 3: unconnected-(RV702-Pad3) -> +3V3
- RV703 pad 1: unconnected-(RV703-Pad1) -> GND
- RV703 pad 2: unconnected-(RV703-Pad2) -> MUX_IO2
- RV703 pad 3: unconnected-(RV703-Pad3) -> +3V3
- RV704 pad 1: unconnected-(RV704-Pad1) -> GND
- RV704 pad 2: unconnected-(RV704-Pad2) -> MUX_IO1
- RV704 pad 3: unconnected-(RV704-Pad3) -> +3V3
- RV705 pad 1: unconnected-(RV705-Pad1) -> GND
- RV705 pad 2: unconnected-(RV705-Pad2) -> MUX_IO7
- RV705 pad 3: unconnected-(RV705-Pad3) -> +3V3
- RV706 pad 1: unconnected-(RV706-Pad1) -> GND
- RV706 pad 2: unconnected-(RV706-Pad2) -> MUX_IO5
- RV706 pad 3: unconnected-(RV706-Pad3) -> +3V3
- RV707 pad 1: unconnected-(RV707-Pad1) -> GND
- RV707 pad 2: unconnected-(RV707-Pad2) -> MUX_IO3
- RV707 pad 3: unconnected-(RV707-Pad3) -> +3V3
- RV708 pad 1: unconnected-(RV708-Pad1) -> GND
- RV708 pad 2: unconnected-(RV708-Pad2) -> MUX_IO0
- RV708 pad 3: unconnected-(RV708-Pad3) -> +3V3
- RV709 pad 1: unconnected-(RV709-Pad1) -> GND
- RV709 pad 2: unconnected-(RV709-Pad2) -> MUX_IO8
- RV709 pad 3: unconnected-(RV709-Pad3) -> +3V3
- RV710 pad 1: unconnected-(RV710-Pad1) -> GND
- RV710 pad 2: unconnected-(RV710-Pad2) -> MUX_IO10
- RV710 pad 3: unconnected-(RV710-Pad3) -> +3V3
- RV711 pad 1: unconnected-(RV711-Pad1) -> GND
- RV711 pad 2: unconnected-(RV711-Pad2) -> MUX_IO12
- RV711 pad 3: unconnected-(RV711-Pad3) -> +3V3
- RV712 pad 1: unconnected-(RV712-Pad1) -> GND
- RV712 pad 2: unconnected-(RV712-Pad2) -> MUX_IO15
- RV712 pad 3: unconnected-(RV712-Pad3) -> +3V3
- RV713 pad 1: unconnected-(RV713-Pad1) -> GND
- RV713 pad 2: unconnected-(RV713-Pad2) -> MUX_IO9
- RV713 pad 3: unconnected-(RV713-Pad3) -> +3V3
- RV714 pad 1: unconnected-(RV714-Pad1) -> GND
- RV714 pad 2: unconnected-(RV714-Pad2) -> MUX_IO11
- RV714 pad 3: unconnected-(RV714-Pad3) -> +3V3
- RV715 pad 1: unconnected-(RV715-Pad1) -> GND
- RV715 pad 2: unconnected-(RV715-Pad2) -> MUX_IO13
- RV715 pad 3: unconnected-(RV715-Pad3) -> +3V3
- RV716 pad 1: unconnected-(RV716-Pad1) -> GND
- RV716 pad 2: unconnected-(RV716-Pad2) -> MUX_IO14
- RV716 pad 3: unconnected-(RV716-Pad3) -> +3V3
- RV717 pad 1: unconnected-(RV717-Pad1) -> GND
- RV717 pad 2: unconnected-(RV717-Pad2) -> VOL
- RV717 pad 3: unconnected-(RV717-Pad3) -> +3V3
- U401 pad 12: IO27/ADCDAT -> IO27/MUX_S1
- U401 pad 14: IO12/MUX_S2 -> IO12/MUX_S0
- U401 pad 24: IO2/MUX_S0 -> IO2/MUX_S2
- U401 pad 26: IO4/MUX_S1 -> IO4/MUX_S3
- U401 pad 29: IO5/SD_CS -> VOL
- U401 pad 30: IO18/SD_CLK -> unconnected-(U401-Pad30)
- U401 pad 31: IO19/SD_MISO -> unconnected-(U401-Pad31)
- U401 pad 37: IO23/SD_MOSI -> unconnected-(U401-Pad37)
- U401 pad 4: I36 -> unconnected-(U401-Pad4)
- U401 pad 5: I39 -> unconnected-(U401-Pad5)
- U401 pad 6: I34 -> unconnected-(U401-Pad6)
- U401 pad 7: I35 -> unconnected-(U401-Pad7)
- U401 pad 8: IO32/MUX_S3 -> unconnected-(U401-Pad8)
- U501 pad 1: LIP -> unconnected-(U501-Pad1)
- U501 pad 19: AUXL -> unconnected-(U501-Pad19)
- U501 pad 2: LIN -> unconnected-(U501-Pad2)
- U501 pad 20: AUXR -> unconnected-(U501-Pad20)
- U501 pad 21: OUT4 -> Line_Out_R
- U501 pad 22: OUT3 -> Line_Out_L
- U501 pad 23: ROUT2 -> unconnected-(U501-Pad23)
- U501 pad 25: LOUT2 -> unconnected-(U501-Pad25)
- U501 pad 29: ROUT1 -> HP_R
- U501 pad 3: L2 -> unconnected-(U501-Pad3)
- U501 pad 30: LOUT1 -> HP_L
- U501 pad 4: RIP -> unconnected-(U501-Pad4)
- U501 pad 5: RIN -> unconnected-(U501-Pad5)
- U501 pad 6: R2 -> unconnected-(U501-Pad6)
- U501 pad 9: IO27/ADCDAT -> unconnected-(U501-Pad9)
- U602 pad 1: MIDI_IN -> MIDI_OUT
- U602 pad 10: OUT -> unconnected-(U602-Pad10)
- U602 pad 11: Net-(U602-Pad11) -> unconnected-(U602-Pad11)
- U602 pad 12: Net-(U602-Pad11) -> unconnected-(U602-Pad12)
- U602 pad 13: MIDI_OUT -> unconnected-(U602-Pad13)
- U602 pad 2: Net-(U602-Pad2) -> unconnected-(U602-Pad2)
- U602 pad 3: Net-(U602-Pad2) -> unconnected-(U602-Pad3)
- U602 pad 4: THRU -> OUT
- U701 pad 10: IO2/MUX_S0 -> IO12/MUX_S0
- U701 pad 11: IO4/MUX_S1 -> IO27/MUX_S1
- U701 pad 13: IO32/MUX_S3 -> IO4/MUX_S3
- U701 pad 14: IO12/MUX_S2 -> IO2/MUX_S2

Commit message: updates
Parts:
- moved SW401 119.9 mm to (195.1, 69.8), turned to -90 degrees
- moved C403 108.1 mm to (187.7, 65.2)
- moved R404 105.8 mm to (184.5, 68.0)
- moved R403 105.2 mm to (184.5, 72.3)
- moved Q401 105.0 mm to (187.6, 68.1)
- moved Q402 105.0 mm to (187.6, 72.4)
- moved RV717 42.4 mm to (132.9, 80.5)
- moved C701 37.6 mm to (142.7, 110.6), turned to 90 degrees
- moved U701 22.4 mm to (135.4, 116.8)
- moved R503 19.7 mm to (120.7, 65.3), turned to -90 degrees
- moved C304 17.6 mm to (169.5, 71.5)
- moved VR302 17.4 mm to (172.6, 71.7), turned to 180 degrees
- moved D402 17.3 mm to (187.2, 54.1)
- moved R301 15.6 mm to (171.5, 75.6), turned to 0 degrees
- moved R302 14.4 mm to (171.5, 74.3), turned to 180 degrees
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Connections:
- net Net-(J401-PadA5) renamed /MCU - USB/CC1
- net Net-(J401-PadB5) renamed /MCU - USB/CC2
- net Net-(R405-Pad2) renamed /MCU - USB/CP2102_VBUS
- net Net-(R407-Pad2) renamed /MCU - USB/CP2102_RST
- D402 pad 2: +5V -> VBUS
- J503 pad 2: unconnected-(J503-Pad2) -> GND
- RV703 pad 2: MUX_IO2 -> MUX_IO3
- RV707 pad 2: MUX_IO3 -> MUX_IO2
- RV711 pad 2: MUX_IO12 -> MUX_IO13
- RV715 pad 2: MUX_IO13 -> MUX_IO12
- U602 pad 2: unconnected-(U602-Pad2) -> Net-(U602-Pad2)
- U602 pad 3: unconnected-(U602-Pad3) -> Net-(U602-Pad2)
Routing:
- net +3V3: track 0.00 -> 817.3 mm, vias 0 -> 13
- net +5V: track 0.00 -> 181.6 mm, vias 0 -> 7
- net /MCU - USB/EN: track 0.00 -> 132.2 mm, vias 0 -> 2
- net IO0/MCLK: track 0.00 -> 130.9 mm
- net IO4/MUX_S3: track 0.00 -> 84.7 mm, vias 0 -> 3
- net IO27/MUX_S1: track 0.00 -> 79.5 mm, vias 0 -> 4
- net MUX_IO14: track 0.00 -> 78.3 mm
- net MUX_IO1: track 0.00 -> 77.4 mm
- net IO2/MUX_S2: track 0.00 -> 71.6 mm
- net IO12/MUX_S0: track 0.00 -> 71.5 mm, vias 0 -> 2
- net MIDI_IN_TIP: track 0.00 -> 68.8 mm, vias 0 -> 2
- net MUX_IO9: track 0.00 -> 65.1 mm
- net MUX_IO6: track 0.00 -> 64.8 mm
- net IO15/MUX_COM: track 0.00 -> 64.7 mm, vias 0 -> 2
- net MUX_IO12: track 0.00 -> 62.3 mm
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- added copper zone on F.Cu, net +3.3VA
- added copper zone on F.Cu, net +3V3
- added copper zone on F.Cu, net +5V
- added copper zone on F.Cu, net /POWER/BUCK1_SW
- added copper zone on F.Cu, net GND
- added copper zone on In1.Cu, net GND
- added copper zone on In2.Cu, net GND
Other:
- copper layers 2 -> 4
- board text added: "3V3 ANALOG"
- board text added: "3V3-DIGI"
- board text added: "AUDIO CODEC"
- board text added: "MIDI"
- board text added: "RST - BOOT"
- board text added: "USB"

Commit message: updates
Parts:
- R603, R604: footprint MY RESISTOR LIBRARY:0805W8F330JT5E -> MY RESISTOR LIBRARY:0603WAF330JT5E
- moved R507 0.10 mm to (101.9, 44.7)
- moved R505 0.09 mm to (116.1, 44.2)
- moved R603 0.08 mm to (172.0, 39.4)
- moved R504 0.07 mm to (101.8, 41.2)
- moved R402 0.06 mm to (182.8, 57.0)
Connections:
- U501 pad 32: MICBIAS -> unconnected-(U501-Pad32)
Routing:
- net +3V3: track 817.3 -> 252.6 mm
- net +5V: track 181.6 -> 186.5 mm
- net IO4/MUX_S3: track 84.7 -> 82.5 mm, vias 3 -> 2
- net IO15/MUX_COM: track 64.7 -> 65.8 mm
- net IO33/BCLK: track 36.2 -> 37.3 mm
- net Line_Out_R: track 55.8 -> 54.8 mm
- net IO21/CODEC_SDIN: track 54.3 -> 55.0 mm
- net IO2/MUX_S2: track 71.6 -> 72.2 mm
- net VBUS: track 23.4 -> 24.0 mm
- net GND: track 50.4 -> 50.7 mm, vias 49 -> 146
- added copper zone on B.Cu, net +3V3

Commit message: updates
Parts:
- added C506: 1u, MY CAPACITOR LIBRARY:CL10A105KB8NNNC_0603, F.Cu at (92.4, 41.2)
- added C507: 1u, MY CAPACITOR LIBRARY:CL10A105KB8NNNC_0603, F.Cu at (105.0, 44.9)
- added H105: MountingHole, MountingHole:MountingHole_2.5mm, F.Cu at (75.2, 37.6)
- added H106: MountingHole, MountingHole:MountingHole_2.5mm, F.Cu at (195.6, 37.6)
- added H107: MountingHole, MountingHole:MountingHole_2.5mm, F.Cu at (195.6, 158.0)
- added H108: MountingHole, MountingHole:MountingHole_2.5mm, F.Cu at (75.2, 158.0)
- added J501: PJ-342B-TX-SMT, MY CONNECTOR LIBRARY:PJ-342B-TX-SMT, F.Cu at (98.9, 40.9)
- added J603: PJ-342B-TX-SMT, MY CONNECTOR LIBRARY:PJ-342B-TX-SMT, F.Cu at (185.4, 40.9)
- added R605: 33R, MY RESISTOR LIBRARY:0603WAF330JT5E, F.Cu at (179.7, 39.6)
- added R606: 33R, MY RESISTOR LIBRARY:0603WAF330JT5E, F.Cu at (191.4, 45.0)
- moved H103 221.0 mm to (40.4, 0.59)
- moved H102 158.1 mm to (40.4, 7.14)
- moved H104 156.4 mm to (33.9, 7.14)
- moved H101 55.5 mm to (33.9, 0.59)
- moved R303 12.3 mm to (193.9, 46.2), turned to 0 degrees
- moved D301 8.34 mm to (193.4, 43.5), turned to 0 degrees
- moved J602 6.93 mm to (171.9, 40.9)
- moved R604 6.91 mm to (178.7, 44.9)
- moved J503 6.56 mm to (85.4, 40.9)
- moved R603 6.14 mm to (165.9, 39.6)
- moved C510 6.07 mm to (104.7, 40.0), turned to 90 degrees
- moved R504 4.58 mm to (106.4, 41.3)
- moved R506 3.66 mm to (117.7, 44.9), turned to -90 degrees
- moved J601 3.66 mm to (158.4, 40.9)
- moved J502 3.65 mm to (112.4, 40.9)
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Connections:
- U401 pad 12: IO27/MUX_S1 -> IO27/ADCDAT
- U401 pad 8: unconnected-(U401-Pad8) -> IO32/MUX_S1
- U501 pad 3: unconnected-(U501-Pad3) -> Line_in_L
- U501 pad 6: unconnected-(U501-Pad6) -> Line_In_R
- U501 pad 9: unconnected-(U501-Pad9) -> IO27/ADCDAT
- U602 pad 10: unconnected-(U602-Pad10) -> THRU
- U602 pad 11: unconnected-(U602-Pad11) -> Net-(U602-Pad11)
- U602 pad 12: unconnected-(U602-Pad12) -> Net-(U602-Pad11)
- U602 pad 13: unconnected-(U602-Pad13) -> MIDI_IN
- U701 pad 11: IO27/MUX_S1 -> IO32/MUX_S1
Routing:
- net IO32/MUX_S1: track 0.00 -> 85.5 mm, vias 0 -> 4
- net IO27/MUX_S1: track 79.4 -> 0.00 mm, vias 4 -> 0
- net THRU: track 0.00 -> 48.3 mm, vias 0 -> 4
- net IO27/ADCDAT: track 0.00 -> 44.4 mm, vias 0 -> 2
- net Line_In_R: track 0.00 -> 32.5 mm, vias 0 -> 4
- net Line_in_L: track 0.00 -> 24.5 mm, vias 0 -> 4
- net +3V3: track 252.6 -> 265.2 mm
- net Line_Out_R: track 54.8 -> 44.9 mm
- net MIDI_IN: track 51.2 -> 60.7 mm
- net OUT: track 44.8 -> 37.6 mm
- net GND: track 50.7 -> 56.4 mm, vias 146 -> 133
- net Net-(U602-Pad11): track 0.00 -> 3.87 mm
- net MIDI_IN_RING: track 45.9 -> 42.3 mm
- net Net-(C506-Pad1): track 0.00 -> 2.87 mm
- net Net-(C508-Pad2): track 16.9 -> 14.2 mm
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Other:
- board text added: "AUDIO DSP PLATFORM"
- board text added: "J.UCEDO V1 Rev0 05-06-23"
- board text added: "SOLAR AUDIO"

Commit message: updates
Parts:
- removed H101, H102, H103, H104: MountingHole, MountingHole:MountingHole_2.5mm_Pad
- moved R506 4.73 mm to (114.5, 48.4), turned to 180 degrees
- moved R507 3.84 mm to (106.6, 44.9), turned to -90 degrees
- moved C510 0.16 mm to (104.6, 39.9)
- moved C511 0.14 mm to (119.0, 45.0)
- moved R504 0.06 mm to (106.4, 41.3)
Routing:
- net Net-(C511-Pad1): track 4.07 -> 10.0 mm
- net MIDI_IN_TIP: track 68.6 -> 71.1 mm
- net Net-(C510-Pad1): track 3.19 -> 4.96 mm
- net GND: track 56.4 -> 55.3 mm, vias 133 -> 132
- net unconnected-(J501-Pad4): track 1.06 -> 0.00 mm, vias 1 -> 0

Commit message: updates
Parts:
- R301: footprint MY RESISTOR LIBRARY:0402WGF1003TCE -> MY RESISTOR LIBRARY:0603WAF1003T5E
- R302: footprint MY RESISTOR LIBRARY:0402WGF2202TCE -> MY RESISTOR LIBRARY:0603WAF2200T5E
- R303: footprint MY RESISTOR LIBRARY:0402WGF2201TCE -> MY RESISTOR LIBRARY:0603WAF2201T5E
- R504, R505: footprint MY RESISTOR LIBRARY:0805W8F1000T5E -> MY RESISTOR LIBRARY:0603WAF1000T5E
- moved C510 10.3 mm to (110.2, 48.5), turned to 0 degrees
- moved RV716 8.06 mm to (186.2, 147.0), turned to 0 degrees
- moved RV712 8.05 mm to (152.3, 147.0), turned to 0 degrees
- moved RV708 8.04 mm to (118.4, 147.0), turned to 0 degrees
- moved RV704 8.03 mm to (84.5, 147.0), turned to 0 degrees
- moved RV715 7.81 mm to (186.2, 126.1), turned to 0 degrees
- moved RV711 7.80 mm to (152.3, 126.1), turned to 0 degrees
- moved RV707 7.79 mm to (118.4, 126.1), turned to 0 degrees
- moved RV703 7.78 mm to (84.5, 126.1), turned to 0 degrees
- moved RV714 7.56 mm to (186.2, 105.2), turned to 0 degrees
- moved RV710 7.55 mm to (152.3, 105.2), turned to 0 degrees
- moved RV706 7.54 mm to (118.4, 105.2), turned to 0 degrees
- moved RV702 7.53 mm to (84.5, 105.2), turned to 0 degrees
- moved RV713 7.31 mm to (186.2, 84.3), turned to 0 degrees
- moved RV709 7.30 mm to (152.3, 84.3), turned to 0 degrees
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Routing:
- net Line_Out_R: track 45.0 -> 32.6 mm, vias 2 -> 4
- net +3V3: track 265.2 -> 275.9 mm, vias 13 -> 12
- net /MCU - USB/EN: track 131.8 -> 121.5 mm
- net Net-(C510-Pad1): track 4.96 -> 10.9 mm
- net THRU: track 48.3 -> 54.0 mm
- net +5V: track 186.5 -> 191.7 mm
- net Line_Out_L: track 21.6 -> 26.0 mm, vias 2 -> 4
- net IO22/CODEC_SCLK: track 54.4 -> 50.1 mm
- net IO27/ADCDAT: track 44.4 -> 47.1 mm
- net HP_R: track 48.2 -> 45.7 mm
- net IO25/LRC: track 32.4 -> 34.2 mm
- net MIDI_IN_TIP: track 71.1 -> 72.4 mm
- net VOL: track 34.9 -> 36.2 mm
- net IO26/DACDAT: track 42.3 -> 43.6 mm
- net IO0/MCLK: track 131.1 -> 132.4 mm
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Other:
- outline, holes or cut-outs redrawn
- board text added: "J.UCEDO V1 Rev0 07-06-23"
- board text removed: "J.UCEDO V1 Rev0 05-06-23"
