File: DESIGN FILES/ESP32 synth.kicad_pcb (KiCad board)
At the start: 4 copper layers, 127 x 127 mm, 97 parts, among them J401 YTC-TC16S-28, J501 PJ-342B-TX-SMT, J502 PJ-342B-TX-SMT, J503 PJ-342B-TX-SMT, J601 PJ-342B-TX-SMT, J602 PJ-342B-TX-SMT, J603 PJ-342B-TX-SMT, Q401 MMBT3904, Q402 MMBT3904, SW401 TS-1187A-B-A-B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

Commit message: up
Parts:
- moved R603 0.29 mm to (165.6, 39.6)
Routing:
- net Line_Out_L: track 26.0 -> 28.1 mm
