File: DESIGN FILES/mcu_usb.kicad_sch (KiCad schematic)
At the start: 26 parts, among them J401 YTC-TC16S-28, Q401 MMBT3904, Q402 MMBT3904, SW401 TS-1187A-B-A-B, U401 ESP32-WROVER-E-N4R8, U402 CP2102N-A02-GQFN28R

Commit message: updates
Parts:
- C401: value 1u -> (none); footprint MY CAPACITOR LIBRARY:CL10A105KB8NNNC_0603 -> (none)
- C402: value 22u -> (none); footprint MY CAPACITOR LIBRARY:0603_CL10A226MQ8NRNC -> (none)
- C403, C404, C407: value 100n -> (none); footprint MY CAPACITOR LIBRARY:CC0603KRX7R9BB104_0603 -> (none)
- C405, C406: value 4.7u -> (none); footprint MY CAPACITOR LIBRARY:CL10A475KO8NNNC_0603 -> (none)
- C408: value 1uF -> (none); footprint MY CAPACITOR LIBRARY:CL10A105KB8NNNC_0603 -> (none)
- D402: value SP0503BAHTG -> (none); footprint MY DIODE LIBRARY:SP0503BAHTG_SOT-143 -> (none)
- F401: value SMD0805P020TF -> (none); footprint MY FUSE LIBRARY:0805_SMD0805P020TF -> (none)
- FB401: value 120R -> (none); footprint MY FERRITE BEAD LIBRARY:0603_BLM18AG121SN1D -> (none)
- J401: value YTC-TC16S-28 -> (none); footprint MY CONNECTOR LIBRARY:YTC-TC16S-28 -> (none)
- Q401, Q402: value MMBT3904 -> (none); footprint MY TRANSISTOR LIBRARY:MMBT3904_SOT-23 -> (none)
- R401, R403, R404: value 10k -> (none); footprint MY RESISTOR LIBRARY:0603WAF1002T5E -> (none)
- R402: value 1.5k -> (none); footprint MY RESISTOR LIBRARY:CQ03WAJ0152T5E -> (none)
- R405: value 22k -> (none); footprint MY RESISTOR LIBRARY:0603WAF2202T5E -> (none)
- R406: value 47k -> (none); footprint MY RESISTOR LIBRARY:0603WAF4702T5E -> (none)
- R407: value 1k -> (none); footprint MY RESISTOR LIBRARY:0603WAF1001T5E -> (none)
- R408, R409: value 5.1k -> (none); footprint MY RESISTOR LIBRARY:0603WAF5101T5E -> (none)
- SW401: value TS-1187A-B-A-B -> (none); footprint MY SWITCH LIBRARY:TS-1187A-B-A-B_smd -> (none)
- U401: value ESP32-WROVER-E-N4R8 -> (none); footprint MY MICROCONTROLLER LIBRARY:XCVR_ESP32-WROVER-E-N4R8 -> (none)
- U402: value CP2102N-A02-GQFN28R -> (none); footprint MY IC LIBRARY:CP2102N-A02-GQFN28R_QFN-28 -> (none)
Connections:
- net I34: no longer names the net of U401.6 (IO34)
- net I35: no longer names the net of U401.7 (IO35)
- net I36: no longer names the net of U401.4 (SENSOR_VP)
- net I39: no longer names the net of U401.5 (SENSOR_VN)
- net IO12/MUX_S2 renamed IO12/MUX_S0
- net IO18/SD_CLK: no longer names the net of U401.30 (IO18)
- net IO19/SD_MISO: no longer names the net of U401.31 (IO19)
- net IO23/SD_MOSI: no longer names the net of U401.37 (IO23)
- net IO27/ADCDAT renamed IO27/MUX_S1
- net IO2/MUX_S0 renamed IO2/MUX_S2
- net IO32/MUX_S3: no longer names the net of U401.8 (IO32)
- net IO4/MUX_S1 renamed IO4/MUX_S3
- net IO5/SD_CS renamed VOL
- no-connect marks 27 -> 50

Commit message: updates
Connections:
- net CC2: now reaches J401.B5 (CC2), R408.1
- net CP2102_VBUS: now reaches R405.2, R406.1, U402.8 (VBUS)
- net CP2102_RST: now reaches R407.2, U402.9 (~{RST})
- net CC1: now reaches J401.A5 (CC1), R409.1
- no-connect marks 50 -> 35
Other:
- note added: "MCU - USB"
- note added: "see datasheet for voltage divider"
- note removed: "DNP"
- company: (none) -> Joël Ucedo
- title: (none) -> ESP32 SYNTH
- moved on the sheet: C401, C402, C403, C404, C405, C406, C407, C408, D402, F401, FB401, J401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

Commit message: updates
Parts:
- C401: value (none) -> 1u; footprint (none) -> MY CAPACITOR LIBRARY:CL10A105KB8NNNC_0603
- C402: value (none) -> 22u; footprint (none) -> MY CAPACITOR LIBRARY:0603_CL10A226MQ8NRNC
- C403, C404, C407: value (none) -> 100n; footprint (none) -> MY CAPACITOR LIBRARY:CC0603KRX7R9BB104_0603
- C405, C406: value (none) -> 4.7u; footprint (none) -> MY CAPACITOR LIBRARY:CL10A475KO8NNNC_0603
- C408: value (none) -> 1uF; footprint (none) -> MY CAPACITOR LIBRARY:CL10A105KB8NNNC_0603
- D402: value (none) -> SP0503BAHTG; footprint (none) -> MY DIODE LIBRARY:SP0503BAHTG_SOT-143
- F401: value (none) -> SMD0805P020TF; footprint (none) -> MY FUSE LIBRARY:0805_SMD0805P020TF
- FB401: value (none) -> 120R; footprint (none) -> MY FERRITE BEAD LIBRARY:0603_BLM18AG121SN1D
- J401: value (none) -> YTC-TC16S-28; footprint (none) -> MY CONNECTOR LIBRARY:YTC-TC16S-28
- Q401, Q402: value (none) -> MMBT3904; footprint (none) -> MY TRANSISTOR LIBRARY:MMBT3904_SOT-23
- R401, R403, R404: value (none) -> 10k; footprint (none) -> MY RESISTOR LIBRARY:0603WAF1002T5E
- R402: value (none) -> 1.5k; footprint (none) -> MY RESISTOR LIBRARY:CQ03WAJ0152T5E
- R405: value (none) -> 22k; footprint (none) -> MY RESISTOR LIBRARY:0603WAF2202T5E
- R406: value (none) -> 47k; footprint (none) -> MY RESISTOR LIBRARY:0603WAF4702T5E
- R407: value (none) -> 1k; footprint (none) -> MY RESISTOR LIBRARY:0603WAF1001T5E
- R408, R409: value (none) -> 5.1k; footprint (none) -> MY RESISTOR LIBRARY:0603WAF5101T5E
- SW401: value (none) -> TS-1187A-B-A-B; footprint (none) -> MY SWITCH LIBRARY:TS-1187A-B-A-B_smd
- U401: value (none) -> ESP32-WROVER-E-N4R8; footprint (none) -> MY MICROCONTROLLER LIBRARY:XCVR_ESP32-WROVER-E-N4R8
- U402: value (none) -> CP2102N-A02-GQFN28R; footprint (none) -> MY IC LIBRARY:CP2102N-A02-GQFN28R_QFN-28
Connections:
- net +5V: no longer D402.2
- net VBUS: now also D402.2

Commit message: updates
Changed lines of the file:
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@@
   (junction (at 356.87 139.7) (diameter 0) (color 0 0 0 0)
   )
+  (junction (at 121.92 175.26) (diameter 0) (color 0 0 0 0)
+  )
   (junction (at 115.57 137.16) (diameter 0) (color 0 0 0 0)
   )
@@
   )
   (junction (at 284.48 217.17) (diameter 0) (color 0 0 0 0)
+  )
+  (junction (at 379.73 76.2) (diameter 0) (color 0 0 0 0)
   )
   (junction (at 68.58 149.86) (diameter 0) (color 0 0 0 0)
@@
     (stroke (width 0) (type default) (color 0 0 0 0))
   )
+  (wire (pts (xy 121.92 175.26) (xy 123.19 175.26))
+    (stroke (width 0) (type default) (color 0 0 0 0))
+  )
   (wire (pts (xy 344.17 144.78) (xy 344.17 151.13))
     (stroke (width 0) (type default) (color 0 0 0 0))
@@
     (stroke (width 0) (type default) (color 0 0 0 0))
   )
+  (wire (pts (xy 379.73 73.66) (xy 379.73 76.2))
+    (stroke (width 0) (type default) (color 0 0 0 0))
+  )
   (wire (pts (xy 275.59 92.71) (xy 275.59 76.2))
     (stroke (width 0) (type default) (color 0 0 0 0))
@@
     (stroke (width 0) (type default) (color 0 0 0 0))
   )
-  (wire (pts (xy 119.38 175.26) (xy 123.19 175.26))
+  (wire (pts (xy 119.38 175.26) (xy 121.92 175.26))
     (stroke (width 0) (type default) (color 0 0 0 0))
   )
@@
   )
   (wire (pts (xy 288.29 209.55) (xy 308.61 209.55))
+    (stroke (width 0) (type default) (color 0 0 0 0))
+  )
+  (wire (pts (xy 121.92 175.26) (xy 121.92 177.8))
     (stroke (width 0) (type default) (color 0 0 0 0))
   )
@@
   (symbol (lib_id "power:VBUS") (at 119.38 175.26 90) (unit 1)
     (in_bom yes) (on_board yes)
-    (property "Reference" "#PWR?" (id 0) (at 123.19 175.26 0)
+    (property "Reference" "#PWR0120" (id 0) (at 123.19 175.26 0)
       (effects (font (size 1.27 1.27)) hide)
     )
@@
     )
     (property "Datasheet" "" (id 3) (at 119.38 175.26 0)
+      (effects (font (size 1.27 1.27)) hide)
+    )
+    (pin "1")
+  )
+  (symbol (lib_id "power:PWR_FLAG") (at 379.73 73.66 0) (unit 1)
+    (in_bom yes) (on_board yes) (fields_autoplaced)
+    (property "Reference" "#FLG0103" (id 0) (at 379.73 71.755 0)
+      (effects (font (size 1.27 1.27)) hide)
+    )
+    (property "Value" "PWR_FLAG" (id 1) (at 379.73 68.58 0))
+    (property "Footprint" "" (id 2) (at 379.73 73.66 0)
+      (effects (font (size 1.27 1.27)) hide)
+    )
+    (property "Datasheet" "~" (id 3) (at 379.73 73.66 0)
       (effects (font (size 1.27 1.27)) hide)
     )
@@
     )
     (pin "1")
-  )
-  (symbol (lib_id "MY RESISTOR LIBRARY:0603WAF5101T5E") (at 95.25 151.13 0) (unit 1)
-    (in_bom yes) (on_board yes) (fields_autoplaced)
-    (property "Reference" "R408" (id 0) (at 97.79 149.8599 0)
-      (effects (font (size 1.27 1.27)) (justify left))
-    )
-    (property "Value" "5.1k" (id 1) (at 97.79 152.3999 0)
-      (effects (font (size 1.27 1.27)) (justify left))
-    )
-    (property "Footprint" "MY RESISTOR LIBRARY:0603WAF5101T5E" (id 2) (at 93.472 151.13 90)
-      (effects (font (size 1.27 1.27)) hide)
-    )
-    (property "Datasheet" "~" (id 3) (at 95.25 151.13 0)
-      (effects (font (size 1.27 1.27)) hide)
-    )
-    (pin "1")
-    (pin "2")
   )
   (symbol (lib_id "power:GND") (at 356.87 142.24 0) (unit 1)
@@
     )
     (property "Datasheet" "~" (id 3) (at 133.35 137.16 0)
-      (effects (font (size 1.27 1.27)) hide)
-    )
-    (pin "1")
-    (pin "2")
-  )
-  (symbol (lib_id "MY RESISTOR LIBRARY:CQ03WAJ0152T5E") (at 74.93 160.02 90) (unit 1)
-    (in_bom yes) (on_board yes)
-    (property "Reference" "R402" (id 0) (at 74.93 157.48 90))
-    (property "Value" "1.5k" (id 1) (at 74.93 162.56 90))
-    (property "Footprint" "MY RESISTOR LIBRARY:CQ03WAJ0152T5E" (id 2) (at 74.93 161.798 90)
-      (effects (font (size 1.27 1.27)) hide)
-    )
-    (property "Datasheet" "~" (id 3) (at 74.93 160.02 0)
       (effects (font (size 1.27 1.27)) hide)
     )
@@
     (pin "1")
   )
-  (symbol (lib_id "MY RESISTOR LIBRARY:0603WAF5101T5E") (at 105.41 151.13 0) (unit 1)
-    (in_bom yes) (on_board yes) (fields_autoplaced)
-    (property "Reference" "R409" (id 0) (at 107.95 149.8599 0)
-      (effects (font (size 1.27 1.27)) (justify left))
-    )
-    (property "Value" "5.1k" (id 1) (at 107.95 152.3999 0)
-      (effects (font (size 1.27 1.27)) (justify left))
-    )
-    (property "Footprint" "MY RESISTOR LIBRARY:0603WAF5101T5E" (id 2) (at 103.632 151.13 90)
-      (effects (font (size 1.27 1.27)) hide)
-    )
-    (property "Datasheet" "~" (id 3) (at 105.41 151.13 0)
-      (effects (font (size 1.27 1.27)) hide)
-    )
-    (pin "1")
-    (pin "2")
-  )
   (symbol (lib_id "MY RESISTOR LIBRARY:0603WAF1002T5E") (at 293.37 217.17 90) (unit 1)
     (in_bom yes) (on_board yes) (fields_autoplaced)
@@
     (pin "2")
   )
+  (symbol (lib_id "power:PWR_FLAG") (at 121.92 177.8 180) (unit 1)
+    (in_bom yes) (on_board yes) (fields_autoplaced)
+    (property "Reference" "#FLG0104" (id 0) (at 121.92 179.705 0)
+      (effects (font (size 1.27 1.27)) hide)
+    )
+    (property "Value" "PWR_FLAG" (id 1) (at 121.92 182.88 0))
+    (property "Footprint" "" (id 2) (at 121.92 177.8 0)
+      (effects (font (size 1.27 1.27)) hide)
+    )
+    (property "Datasheet" "~" (id 3) (at 121.92 177.8 0)
+      (effects (font (size 1.27 1.27)) hide)
+    )
+    (pin "1")
+  )
   (symbol (lib_id "power:GND") (at 215.9 115.57 0) (unit 1)
     (in_bom yes) (on_board yes) (fields_autoplaced)
@@
     )
     (pin "1")
+  )
+  (symbol (lib_id "MY RESISTOR LIBRARY:0603WAF5101T5E") (at 105.41 151.13 0) (unit 1)
+    (in_bom yes) (on_board yes) (fields_autoplaced)
+    (property "Reference" "R409" (id 0) (at 107.95 149.8599 0)
+      (effects (font (size 1.27 1.27)) (justify left))
+    )
+    (property "Value" "5.1k" (id 1) (at 107.95 152.3999 0)
+      (effects (font (size 1.27 1.27)) (justify left))
+    )
+    (property "Footprint" "MY RESISTOR LIBRARY:0603WAF5101T5E" (id 2) (at 103.632 151.13 90)
+      (effects (font (size 1.27 1.27)) hide)
+    )
+    (property "Datasheet" "~" (id 3) (at 105.41 151.13 0)
+      (effects (font (size 1.27 1.27)) hide)
+    )
+    (pin "1")
+    (pin "2")
   )
   (symbol (lib_id "power:GND") (at 156.21 157.48 0) (unit 1)
@@
     (pin "1")
   )
+  (symbol (lib_id "MY RESISTOR LIBRARY:CQ03WAJ0152T5E") (at 74.93 160.02 90) (unit 1)
+    (in_bom yes) (on_board yes)
+    (property "Reference" "R402" (id 0) (at 74.93 157.48 90))
+    (property "Value" "1.5k" (id 1) (at 74.93 162.56 90))
+    (property "Footprint" "MY RESISTOR LIBRARY:CQ03WAJ0152T5E" (id 2) (at 74.93 161.798 90)
+      (effects (font (size 1.27 1.27)) hide)
+    )
+    (property "Datasheet" "~" (id 3) (at 74.93 160.02 0)
+      (effects (font (size 1.27 1.27)) hide)
+    )
+    (pin "1")
+    (pin "2")
+  )
   (symbol (lib_id "power:GND") (at 264.16 104.14 0) (unit 1)
     (in_bom yes) (on_board yes) (fields_autoplaced)
@@
     (pin "1")
   )
+  (symbol (lib_id "MY RESISTOR LIBRARY:0603WAF5101T5E") (at 95.25 151.13 0) (unit 1)
+    (in_bom yes) (on_board yes) (fields_autoplaced)
+    (property "Reference" "R408" (id 0) (at 97.79 149.8599 0)
+      (effects (font (size 1.27 1.27)) (justify left))
+    )
+    (property "Value" "5.1k" (id 1) (at 97.79 152.3999 0)
+      (effects (font (size 1.27 1.27)) (justify left))
+    )
+    (property "Footprint" "MY RESISTOR LIBRARY:0603WAF5101T5E" (id 2) (at 93.472 151.13 90)
+      (effects (font (size 1.27 1.27)) hide)
+    )
+    (property "Datasheet" "~" (id 3) (at 95.25 151.13 0)
+      (effects (font (size 1.27 1.27)) hide)
+    )
+    (pin "1")
+    (pin "2")
+  )
   (symbol (lib_id "power:GND") (at 46.99 180.34 0) (unit 1)

Commit message: updates
Connections:
- net IO32/MUX_S1: now reaches U401.8 (IO32)
- net IO27/MUX_S1 renamed IO27/ADCDAT
- no-connect marks 35 -> 34
Changed lines of the file:
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@@
   (no_connect (at 339.09 135.89))
   (no_connect (at 339.09 120.65))
-  (no_connect (at 339.09 106.68))
   (no_connect (at 339.09 88.9))
   (no_connect (at 339.09 96.52))
@@
     (stroke (width 0) (type default) (color 0 0 0 0))
   )
+  (wire (pts (xy 339.09 106.68) (xy 344.17 106.68))
+    (stroke (width 0) (type default) (color 0 0 0 0))
+  )
   (polyline (pts (xy 392.43 63.5) (xy 392.43 158.75))
     (stroke (width 0.5) (type default) (color 0 0 0 0))
@@
     )
   )
+  (global_label "IO32{slash}MUX_S1" (shape input) (at 344.17 106.68 0) (fields_autoplaced)
+    (effects (font (size 1.27 1.27) (thickness 0.254) bold italic) (justify left))
+    (property "Intersheet References" "${INTERSHEET_REFS}" (id 0) (at 360.0919 106.553 0)
+      (effects (font (size 1.27 1.27) (thickness 0.254) bold italic) (justify left) hide)
+    )
+  )
   (global_label "IO0{slash}MCLK" (shape input) (at 297.18 99.06 180) (fields_autoplaced)
     (effects (font (size 1.27 1.27) (thickness 0.254) bold italic) (justify right))
@@
     )
   )
-  (global_label "IO27{slash}MUX_S1" (shape input) (at 344.17 104.14 0) (fields_autoplaced)
+  (global_label "IO27{slash}ADCDAT" (shape input) (at 344.17 104.14 0) (fields_autoplaced)
     (effects (font (size 1.27 1.27) (thickness 0.254) bold italic) (justify left))
-    (property "Intersheet References" "${INTERSHEET_REFS}" (id 0) (at 360.0919 104.013 0)
+    (property "Intersheet References" "${INTERSHEET_REFS}" (id 0) (at 359.6686 104.013 0)
       (effects (font (size 1.27 1.27) (thickness 0.254) bold italic) (justify left) hide)
     )

Commit message: updates
Other:
- note added: "USB-C CIRCUIT & USB > UART CONVERTER"
- note removed: "USB TO UART CONVERTER"
Changed lines of the file:
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@@
     (stroke (width 0) (type default) (color 0 0 0 0))
   )
-  (text "USB TO UART CONVERTER" (at 26.67 63.5 0)
+  (text "USB-C CIRCUIT & USB > UART CONVERTER" (at 26.67 63.5 0)
     (effects (font (size 5 5) bold italic) (justify left bottom))
   )
