File: DESIGN FILES/power.kicad_sch (KiCad schematic)
At the start: 0 parts

Commit message: updates
Parts:
- added C?: 100nF, soundsom:CC0603KRX7R9BB104_0603, symbol soundsom:CC0603KRX7R9BB104
- added C? (x3): 22uF, soundsom:CL10A226MQ8NRNC_0603, symbol soundsom:CL10A226MQ8NRNC
- added C?: 1uF, soundsom:CL10A105KB8NNNC_0603, symbol soundsom:CL10A105KB8NNNC
- added C?: 10uF, soundsom:CL10A106MA8NRNC_0603, symbol soundsom:CL10A106MA8NRNC
- added C?: 22pF, soundsom:CL10C220JB8NNNC_0603, symbol soundsom:CL10C220JB8NNNC
- added L?: 2.2uH, soundsom:CD32YP0302-2R2M_SMD3.5x3x2.1mm, symbol soundsom:CD32YP0302-2R2M
- added R?: 100k, soundsom:0603WAF1003T5E_0603, symbol soundsom:0603WAF1003T5E
- added R?: 22k, soundsom:0603WAF2202T5E_0603, symbol soundsom:0603WAF2202T5E
- added VR?: SY8089AAAC, soundsom:SY8089AAAC_SOT-23-5, symbol soundsom:SY8089AAAC
- added VR?: TPS79333DBVR, soundsom:TPS79333DBVR_SOT-23-5, symbol soundsom:TPS79333DBVR
Connections:
- new net: C?.1, VR?.4 (NR)
- new net: L?.1, VR?.3 (LX)
- new net: C?.2, R?.1, R?.2, VR?.5 (FB)
- new net +3.3VA: C?.1, VR?.5 (OUT)
- new net +3V3: C?.1, C?.1, C?.1, L?.2, R?.1
- new net +5V: C?.1, C?.1, VR?.1 (EN), VR?.1 (IN), VR?.3 (EN), VR?.4 (IN)
- new net GND: C?.2, C?.2, C?.2, C?.2, C?.2, C?.2, R?.2, VR?.2 (GND), VR?.2 (GND)
Other:
- note added: "+5V USB > + 3V3 ANALOG"
- note added: "+5V USB > +3V3 DIGITAL"
- note added: "200mA Low-Noise High PSRR LDO"
- note added: "Buck converter : 2A continuous, 3A peak"
- note added: "Only for audio codec analog part"
- note added: "Vout = 0.6 * (1 + R1/R2)"

Commit message: updates
Parts:
- removed C?: 100nF, soundsom:CC0603KRX7R9BB104_0603, symbol soundsom:CC0603KRX7R9BB104
- removed C? (x3): 22uF, soundsom:CL10A226MQ8NRNC_0603, symbol soundsom:CL10A226MQ8NRNC
- removed C?: 1uF, soundsom:CL10A105KB8NNNC_0603, symbol soundsom:CL10A105KB8NNNC
- removed C?: 10uF, soundsom:CL10A106MA8NRNC_0603, symbol soundsom:CL10A106MA8NRNC
- removed C?: 22pF, soundsom:CL10C220JB8NNNC_0603, symbol soundsom:CL10C220JB8NNNC
- removed L?: 2.2uH, soundsom:CD32YP0302-2R2M_SMD3.5x3x2.1mm, symbol soundsom:CD32YP0302-2R2M
- removed R?: 100k, soundsom:0603WAF1003T5E_0603, symbol soundsom:0603WAF1003T5E
- removed R?: 22k, soundsom:0603WAF2202T5E_0603, symbol soundsom:0603WAF2202T5E
- removed VR?: SY8089AAAC, soundsom:SY8089AAAC_SOT-23-5, symbol soundsom:SY8089AAAC
- removed VR?: TPS79333DBVR, soundsom:TPS79333DBVR_SOT-23-5, symbol soundsom:TPS79333DBVR
- added C301: 1u, MY CAPACITOR LIBRARY:CL10A105KB8NNNC_0603, symbol MY CAPACITOR LIBRARY:CL10A105KB8NNNC
- added C302: 100n, MY CAPACITOR LIBRARY:CC0603KRX7R9BB104_0603, symbol MY CAPACITOR LIBRARY:CC0603KRX7R9BB104
- added C303: 10u, MY CAPACITOR LIBRARY:0603_CL10A106KP8NNNC, symbol MY CAPACITOR LIBRARY:CL10A106KP8NNNC
- added C304: 22u, MY CAPACITOR LIBRARY:0603_CL10A226MQ8NRNC, symbol MY CAPACITOR LIBRARY:CL10A226MQ8NRNC
- added C305: 10u, MY CAPACITOR LIBRARY:CL10A106MA8NRNC_0603, symbol MY CAPACITOR LIBRARY:CL10A106MA8NRNC
- added D301: LED, MY LED LIBRARY:LED_D3.0mm, symbol MY LED LIBRARY:LED
- added L301: 2.2u, MY INDUCTOR LIBRARY:CD32YP0302-2R2M, symbol MY INDUCTOR LIBRARY:CD32YP0302-2R2M
- added R301: 100k, MY RESISTOR LIBRARY:0402WGF1003TCE, symbol MY RESISTOR LIBRARY:0603WAF1003T5E
- added R302: 22k, MY RESISTOR LIBRARY:0402WGF2202TCE, symbol MY RESISTOR LIBRARY:0603WAF2202T5E
- added R303: 2.2k, MY RESISTOR LIBRARY:0402WGF2201TCE, symbol MY RESISTOR LIBRARY:0603WAF2201T5E
- added VR301: TPS79333DBVR, MY REGULATOR LIBRARY:TPS79333DBVR_SOT-23-5, symbol MY REGULATOR LIBRARY:TPS79333DBVR
- added VR302: TLV62569DBV, MY REGULATOR LIBRARY:TLV62569DBVR, symbol MY REGULATOR LIBRARY:TLV62569DBV
Connections:
- net +3.3VA: now also C303.1, VR301.5 (OUT)
- net +3V3: now also C305.1, D301.2 (A), L301.2, R301.1
- net +5V: now also C301.1, C304.1, VR301.1 (IN), VR301.3 (EN), VR302.1 (EN), VR302.4 (VIN)
- net GND: now also C301.2, C302.2, C303.2, C304.2, C305.2, R302.2, R303.2, VR301.2 (GND), VR302.2 (GND)
- new net BUCK1_FB: R301.2, R302.1, VR302.5 (FB)
- new net BUCK1_SW: L301.1, VR302.3 (SW)
- new net LDO_NR: C302.1, VR301.4 (NR)
- new net LED_PWR_K: D301.1 (K), R303.1
Other:
- note added: "+5V > +3V3 ANALOG"
- note added: "+5V > +3V3 DIGITAL"
- note added: "LP Fc = 34KHz"
- note added: "Only for analog audio circuit"
- note added: "V(out) = 0.6*(1+100k/22k) =3.327V"
- note removed: "+5V USB > + 3V3 ANALOG"
- note removed: "+5V USB > +3V3 DIGITAL"
- note removed: "200mA Low-Noise High PSRR LDO"
- note removed: "Buck converter : 2A continuous, 3A peak"
- note removed: "Only for audio codec analog part"
- note removed: "Vout = 0.6 * (1 + R1/R2)"

Commit message: updates
Changed lines of the file:
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@@
   (junction (at 104.14 50.8) (diameter 0) (color 0 0 0 0)
   )
-  (junction (at 58.42 50.8) (diameter 0) (color 0 0 0 0)
-  )
   (junction (at 125.73 50.8) (diameter 0) (color 0 0 0 0)
   )
@@
   (junction (at 55.88 133.35) (diameter 0) (color 0 0 0 0)
   )
+  (junction (at 59.69 50.8) (diameter 0) (color 0 0 0 0)
+  )
   (junction (at 66.04 133.35) (diameter 0) (color 0 0 0 0)
   )
@@
     (stroke (width 0) (type default) (color 0 0 0 0))
   )
-  (wire (pts (xy 58.42 50.8) (xy 58.42 53.34))
-    (stroke (width 0) (type default) (color 0 0 0 0))
-  )
   (wire (pts (xy 101.6 130.81) (xy 101.6 133.35))
     (stroke (width 0) (type default) (color 0 0 0 0))
@@
     (stroke (width 0) (type default) (color 0 0 0 0))
   )
+  (wire (pts (xy 59.69 53.34) (xy 59.69 50.8))
+    (stroke (width 0) (type default) (color 0 0 0 0))
+  )
   (wire (pts (xy 90.17 138.43) (xy 90.17 140.97))
     (stroke (width 0) (type default) (color 0 0 0 0))
@@
     (stroke (width 0) (type default) (color 0 0 0 0))
   )
+  (wire (pts (xy 62.23 53.34) (xy 59.69 53.34))
+    (stroke (width 0) (type default) (color 0 0 0 0))
+  )
   (wire (pts (xy 77.47 53.34) (xy 90.17 53.34))
     (stroke (width 0) (type default) (color 0 0 0 0))
   )
-  (wire (pts (xy 66.04 130.81) (xy 66.04 133.35))
-    (stroke (width 0) (type default) (color 0 0 0 0))
-  )
   (polyline (pts (xy 127 114.3) (xy 127 166.37))
     (stroke (width 0.5) (type default) (color 0 0 0 0))
   )
-  (wire (pts (xy 58.42 53.34) (xy 62.23 53.34))
-    (stroke (width 0) (type default) (color 0 0 0 0))
-  )
   (wire (pts (xy 90.17 53.34) (xy 90.17 67.31))
     (stroke (width 0) (type default) (color 0 0 0 0))
@@
     (stroke (width 0) (type default) (color 0 0 0 0))
   )
-  (wire (pts (xy 45.72 50.8) (xy 58.42 50.8))
+  (wire (pts (xy 59.69 50.8) (xy 62.23 50.8))
     (stroke (width 0) (type default) (color 0 0 0 0))
   )
@@
     (stroke (width 0) (type default) (color 0 0 0 0))
   )
-  (wire (pts (xy 58.42 50.8) (xy 62.23 50.8))
+  (wire (pts (xy 45.72 50.8) (xy 59.69 50.8))
     (stroke (width 0) (type default) (color 0 0 0 0))
   )
@@
     (pin "2")
   )
-  (symbol (lib_id "power:PWR_FLAG") (at 66.04 130.81 0) (unit 1)
-    (in_bom yes) (on_board yes) (fields_autoplaced)
-    (property "Reference" "#FLG0101" (id 0) (at 66.04 128.905 0)
-      (effects (font (size 1.27 1.27)) hide)
-    )
-    (property "Value" "PWR_FLAG" (id 1) (at 66.04 125.73 0))
-    (property "Footprint" "" (id 2) (at 66.04 130.81 0)
-      (effects (font (size 1.27 1.27)) hide)
-    )
-    (property "Datasheet" "~" (id 3) (at 66.04 130.81 0)
-      (effects (font (size 1.27 1.27)) hide)
-    )
-    (pin "1")
-  )
   (symbol (lib_id "MY REGULATOR LIBRARY:TLV62569DBV") (at 69.85 53.34 0) (unit 1)
     (in_bom yes) (on_board yes) (fields_autoplaced)
@@
   (symbol (lib_id "MY CAPACITOR LIBRARY:CC0603KRX7R9BB104") (at 90.17 144.78 0) (unit 1)
     (in_bom yes) (on_board yes)
-    (property "Reference" "C302" (id 0) (at 82.55 143.51 0)
-      (effects (font (size 1.27 1.27)) (justify left))
-    )
-    (property "Value" "100n" (id 1) (at 82.55 146.05 0)
-      (effects (font (size 1.27 1.27)) (justify left))
-    )
+    (property "Reference" "C302" (id 0) (at 81.28 143.51 0)
+      (effects (font (size 1.27 1.27)) (justify left))
+    )
+    (property "Value" "100n" (id 1) (at 81.28 146.05 0)
+      (effects (font (size 1.27 1.27)) (justify left))
+    )

Commit message: updates
Other:
- note added: "POWER"
- company: (none) -> Joël Ucedo
- title: (none) -> ESP32 SYNTH
- moved on the sheet: C301, C302, C303, C304, C305, D301, L301, R301, R302, R303, VR301, VR302

Commit message: updates
Changed lines of the file:
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@@
   (junction (at 125.73 101.6) (diameter 0) (color 0 0 0 0)
   )
+  (junction (at 69.85 115.57) (diameter 0) (color 0 0 0 0)
+  )
   (junction (at 254 95.25) (diameter 0) (color 0 0 0 0)
   )
@@
   (junction (at 114.3 118.11) (diameter 0) (color 0 0 0 0)
   )
+  (junction (at 54.61 101.6) (diameter 0) (color 0 0 0 0)
+  )
   (wire (pts (xy 138.43 118.11) (xy 138.43 120.65))
     (stroke (width 0) (type default) (color 0 0 0 0))
   )
+  (wire (pts (xy 54.61 99.06) (xy 54.61 101.6))
+    (stroke (width 0) (type default) (color 0 0 0 0))
+  )
   (polyline (pts (xy 25.4 76.2) (xy 25.4 139.7))
     (stroke (width 0.5) (type default) (color 0 0 0 0))
@@
     (stroke (width 0) (type default) (color 0 0 0 0))
   )
-  (wire (pts (xy 69.85 111.76) (xy 69.85 120.65))
+  (wire (pts (xy 69.85 111.76) (xy 69.85 115.57))
     (stroke (width 0) (type default) (color 0 0 0 0))
   )
@@
     (stroke (width 0) (type default) (color 0 0 0 0))
   )
+  (wire (pts (xy 69.85 115.57) (xy 69.85 120.65))
+    (stroke (width 0) (type default) (color 0 0 0 0))
+  )
+  (wire (pts (xy 54.61 101.6) (xy 59.69 101.6))
+    (stroke (width 0) (type default) (color 0 0 0 0))
+  )
   (wire (pts (xy 254 95.25) (xy 254 102.87))
     (stroke (width 0) (type default) (color 0 0 0 0))
@@
     (stroke (width 0) (type default) (color 0 0 0 0))
   )
-  (wire (pts (xy 45.72 101.6) (xy 59.69 101.6))
+  (wire (pts (xy 45.72 101.6) (xy 54.61 101.6))
     (stroke (width 0) (type default) (color 0 0 0 0))
   )
@@
   )
   (wire (pts (xy 218.44 95.25) (xy 222.25 95.25))
+    (stroke (width 0) (type default) (color 0 0 0 0))
+  )
+  (wire (pts (xy 69.85 115.57) (xy 74.93 115.57))
     (stroke (width 0) (type default) (color 0 0 0 0))
   )
@@
     (pin "2")
   )
+  (symbol (lib_id "power:PWR_FLAG") (at 74.93 115.57 270) (unit 1)
+    (in_bom yes) (on_board yes) (fields_autoplaced)
+    (property "Reference" "#FLG0102" (id 0) (at 76.835 115.57 0)
+      (effects (font (size 1.27 1.27)) hide)
+    )
+    (property "Value" "PWR_FLAG" (id 1) (at 78.74 115.5699 90)
+      (effects (font (size 1.27 1.27)) (justify left))
+    )
+    (property "Footprint" "" (id 2) (at 74.93 115.57 0)
+      (effects (font (size 1.27 1.27)) hide)
+    )
+    (property "Datasheet" "~" (id 3) (at 74.93 115.57 0)
+      (effects (font (size 1.27 1.27)) hide)
+    )
+    (pin "1")
+  )
   (symbol (lib_id "power:GND") (at 208.28 113.03 0) (unit 1)
     (in_bom yes) (on_board yes) (fields_autoplaced)
@@
       (effects (font (size 1.27 1.27)) hide)
     )
+    (pin "1")
+  )
+  (symbol (lib_id "power:PWR_FLAG") (at 54.61 99.06 0) (unit 1)
+    (in_bom yes) (on_board yes) (fields_autoplaced)
+    (property "Reference" "#FLG0101" (id 0) (at 54.61 97.155 0)
+      (effects (font (size 1.27 1.27)) hide)
+    )
+    (property "Value" "PWR_FLAG" (id 1) (at 54.61 93.98 0))
+    (property "Footprint" "" (id 2) (at 54.61 99.06 0)
+      (effects (font (size 1.27 1.27)) hide)
+    )
+    (property "Datasheet" "~" (id 3) (at 54.61 99.06 0)
+      (effects (font (size 1.27 1.27)) hide)
+    )

Commit message: updates
Parts:
- R301: footprint MY RESISTOR LIBRARY:0402WGF1003TCE -> MY RESISTOR LIBRARY:0603WAF1003T5E
- R302: footprint MY RESISTOR LIBRARY:0402WGF2202TCE -> MY RESISTOR LIBRARY:0603WAF2200T5E
- R303: footprint MY RESISTOR LIBRARY:0402WGF2201TCE -> MY RESISTOR LIBRARY:0603WAF2201T5E
Changed lines of the file:
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@@
       (effects (font (size 1.27 1.27)) (justify left))
     )
-    (property "Footprint" "MY RESISTOR LIBRARY:0402WGF2201TCE" (id 2) (at 136.652 110.49 90)
+    (property "Footprint" "MY RESISTOR LIBRARY:0603WAF2201T5E" (id 2) (at 136.652 110.49 90)
       (effects (font (size 1.27 1.27)) hide)
     )
@@
     (property "Reference" "R302" (id 0) (at 125.73 115.57 90))
     (property "Value" "22k" (id 1) (at 125.73 120.65 90))
-    (property "Footprint" "MY RESISTOR LIBRARY:0402WGF2202TCE" (id 2) (at 125.73 119.888 90)
+    (property "Footprint" "MY RESISTOR LIBRARY:0603WAF2200T5E" (id 2) (at 125.73 119.888 90)
       (effects (font (size 1.27 1.27)) hide)
     )
@@
       (effects (font (size 1.27 1.27)) (justify left))
     )
-    (property "Footprint" "MY RESISTOR LIBRARY:0402WGF1003TCE" (id 2) (at 112.522 110.49 90)
+    (property "Footprint" "MY RESISTOR LIBRARY:0603WAF1003T5E" (id 2) (at 112.522 110.49 90)
       (effects (font (size 1.27 1.27)) hide)
     )
